File: synth/synth.kicad_pcb (KiCad board)
At the start: 2 copper layers, 51 parts, among them J2 10118194-0001LF, U1 ATSAME53N19A, U2 DRA818_iCE40-UP5K-SG48, U4 LMS33460, U5 TPS62120DCNR, U6 BQ24074, U7 DSC6003JI2A, U8 TPS63031

Commit message: Stream 20210528 progress checkpoint.
Parts:
- removed the C2 at (65.8, 63.8)
- added C2: 10uF_10V_0805, up5k-synth:C_0805_2012Metric_Pad1.18x1.45mm_HandSolder, F.Cu at (176.5, 16.0)
- added C2: 1.0uF_10V_0805, up5k-synth:C_0805_2012Metric_Pad1.18x1.45mm_HandSolder, F.Cu at (189.5, 18.5)
- added C24: 0.1uF_10V_0603, up5k-synth:C_0603_1608Metric_Pad1.08x0.95mm_HandSolder, F.Cu at (168.4, 51.0)
- added C4: 10uF_10V_0805, up5k-synth:C_0805_2012Metric_Pad1.18x1.45mm_HandSolder, F.Cu at (181.3, 16.0)
- added J1: MEM2061-01-188-00-A, up5k-synth:MEM2061-01-188-00-A, F.Cu at (192.0, 41.0)
- added J3: PMOD_conn, up5k-synth:PinHeader_2x06_P2.54mm_Horizontal, F.Cu at (46.5, 38.5)
- added L2: Inductance, up5k-synth:LPS3015, F.Cu at (205.5, 15.5)
- added R15: 100kR_4xArray, up5k-synth:R_Array_Convex_4x1206, F.Cu at (176.0, 35.5)
- added R16: 10kR, up5k-synth:R_0805_2012Metric_Pad1.20x1.40mm_HandSolder, F.Cu at (169.5, 28.5)
- added R17: 10kR, up5k-synth:R_0805_2012Metric_Pad1.20x1.40mm_HandSolder, F.Cu at (169.5, 31.4)
- added R18: 10kR, up5k-synth:R_0805_2012Metric_Pad1.20x1.40mm_HandSolder, F.Cu at (174.2, 28.5)
- moved R8 182.9 mm to (236.0, 90.5)
- moved R11 182.1 mm to (245.0, 87.5)
- moved R10 181.1 mm to (230.5, 8.00), turned to 90 degrees
- moved R7 179.8 mm to (229.0, 85.5)
- moved C23 171.7 mm to (217.5, 21.5)
- moved R13 164.2 mm to (216.0, 7.50), turned to 270 degrees
- moved R12 163.7 mm to (220.0, 4.00)
- moved C16 163.4 mm to (236.0, 88.0)
- moved R3 161.5 mm to (232.5, 14.5), turned to 90 degrees
- moved R9 157.2 mm to (240.5, 88.0), turned to 90 degrees
- moved C19 157.0 mm to (221.0, 17.5)
- moved C20 153.7 mm to (219.5, 9.00), turned to 270 degrees
- moved C22 143.4 mm to (216.5, 17.5)
- moved R5 141.0 mm to (221.0, 57.5)
- moved C21 138.4 mm to (206.5, 21.0), turned to 90 degrees
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Connections:
- C9 pad 1: +3V3 -> /mcu_core

Commit message: Project checkpoint on 20210604
Parts:
- added ENC1: rot_encoder_switch, up5k-synth:PEC12R-4xxxF-Sxx, F.Cu at (54.5, 53.5)
- added ENC2: rot_encoder_switch, up5k-synth:PEC12R-4xxxF-Sxx, F.Cu at (36.5, 64.5)
- added J5: AudioJack3_SwitchTR, up5k-synth:STX-3120-5B-577C, F.Cu at (34.5, 49.5)
- added J6: AudioJack3_SwitchTR, up5k-synth:STX-3120-5B-577C, F.Cu at (111.5, -11.5)
- added R19: 360kR, up5k-synth:R_0805_2012Metric_Pad1.20x1.40mm_HandSolder, F.Cu at (89.0, 6.83)
- added R20: 360kR, up5k-synth:R_0805_2012Metric_Pad1.20x1.40mm_HandSolder, F.Cu at (107.4, 3.07)
- added R21: 360kR, up5k-synth:R_0805_2012Metric_Pad1.20x1.40mm_HandSolder, F.Cu at (93.8, 6.83)
- added R22: 360kR, up5k-synth:R_0805_2012Metric_Pad1.20x1.40mm_HandSolder, F.Cu at (98.5, 6.83)
- added R23: 360kR, up5k-synth:R_0805_2012Metric_Pad1.20x1.40mm_HandSolder, F.Cu at (103.3, 6.83)
- added R24: 360kR, up5k-synth:R_0805_2012Metric_Pad1.20x1.40mm_HandSolder, F.Cu at (108.0, 6.02)
- added R25: 360kR, up5k-synth:R_0805_2012Metric_Pad1.20x1.40mm_HandSolder, F.Cu at (112.8, 4.93)
- added R26: 360kR, up5k-synth:R_0805_2012Metric_Pad1.20x1.40mm_HandSolder, F.Cu at (122.6, 3.52)
- added R27: 1kR, up5k-synth:R_0805_2012Metric_Pad1.20x1.40mm_HandSolder, F.Cu at (69.5, 57.0)
- added R28: 1kR, up5k-synth:R_0805_2012Metric_Pad1.20x1.40mm_HandSolder, F.Cu at (69.5, 60.0)
- added R29: 1kR, up5k-synth:R_0805_2012Metric_Pad1.20x1.40mm_HandSolder, F.Cu at (74.2, 57.0)
- added R30: 1kR, up5k-synth:R_0805_2012Metric_Pad1.20x1.40mm_HandSolder, F.Cu at (69.5, 62.9)
- added R31: 1kR, up5k-synth:R_0805_2012Metric_Pad1.20x1.40mm_HandSolder, F.Cu at (74.2, 60.0)
- added R32: 1kR, up5k-synth:R_0805_2012Metric_Pad1.20x1.40mm_HandSolder, F.Cu at (79.0, 57.0)
- added R33: 1kR, up5k-synth:R_0805_2012Metric_Pad1.20x1.40mm_HandSolder, F.Cu at (69.5, 65.8)
- added R34: 1kR, up5k-synth:R_0805_2012Metric_Pad1.20x1.40mm_HandSolder, F.Cu at (74.2, 62.9)
- added R35: 1kR, up5k-synth:R_0805_2012Metric_Pad1.20x1.40mm_HandSolder, F.Cu at (79.0, 60.0)
- added R36: 1kR, up5k-synth:R_0805_2012Metric_Pad1.20x1.40mm_HandSolder, F.Cu at (69.5, 68.8)
- added R37: 1kR, up5k-synth:R_0805_2012Metric_Pad1.20x1.40mm_HandSolder, F.Cu at (83.8, 57.0)
- added R38: 1kR, up5k-synth:R_0805_2012Metric_Pad1.20x1.40mm_HandSolder, F.Cu at (74.2, 65.8)
- added R39: 1kR, up5k-synth:R_0805_2012Metric_Pad1.20x1.40mm_HandSolder, F.Cu at (79.0, 62.9)
- added R40: 1kR, up5k-synth:R_0805_2012Metric_Pad1.20x1.40mm_HandSolder, F.Cu at (83.8, 60.0)
- added R41: 1kR, up5k-synth:R_0805_2012Metric_Pad1.20x1.40mm_HandSolder, F.Cu at (74.2, 68.8)
- added R42: 1kR, up5k-synth:R_0805_2012Metric_Pad1.20x1.40mm_HandSolder, F.Cu at (88.5, 57.0)
- added R43: 1kR, up5k-synth:R_0805_2012Metric_Pad1.20x1.40mm_HandSolder, F.Cu at (79.0, 65.8)
- added R44: 1kR, up5k-synth:R_0805_2012Metric_Pad1.20x1.40mm_HandSolder, F.Cu at (83.8, 62.9)
- added R45: 1kR, up5k-synth:R_0805_2012Metric_Pad1.20x1.40mm_HandSolder, F.Cu at (88.5, 60.0)
- added R46: 1kR, up5k-synth:R_0805_2012Metric_Pad1.20x1.40mm_HandSolder, F.Cu at (79.0, 68.8)
- added R47: 1kR, up5k-synth:R_0805_2012Metric_Pad1.20x1.40mm_HandSolder, F.Cu at (83.8, 65.8)
- added R48: 1kR, up5k-synth:R_0805_2012Metric_Pad1.20x1.40mm_HandSolder, F.Cu at (88.5, 62.9)
- added R49: 1kR, up5k-synth:R_0805_2012Metric_Pad1.20x1.40mm_HandSolder, F.Cu at (83.8, 68.8)
- added R50: 1kR, up5k-synth:R_0805_2012Metric_Pad1.20x1.40mm_HandSolder, F.Cu at (88.5, 65.8)
- added U10: AD8531, up5k-synth:SOIC-8_W3.9mm, F.Cu at (117.0, -0.77)
- added U11: AD8531, up5k-synth:SOIC-8_W3.9mm, F.Cu at (123.4, -2.18)
- added U3: DS1881, up5k-synth:TSSOP-16_4.4x5mm_P0.65mm, F.Cu at (109.4, -1.70)
- added U9: DS1881, up5k-synth:TSSOP-16_4.4x5mm_P0.65mm, F.Cu at (122.4, -9.70)
- moved U1 0.50 mm to (167.5, 62.5), turned to 0 degrees
Connections:
- U1 pad 89: Net-(C7-Pad1) -> /mcu_core
- U2 pad 37: /PDM_L -> /PDM0_L
- U2 pad 38: /PDM_R -> /PDM0_R
- U2 pad 42: Net-(U2-Pad42) -> /PDM1_L
- U2 pad 43: Net-(U2-Pad43) -> /PDM1_R

Commit message: Design checkpoint at 20210609
Parts:
- added C25: CP_10uF_10v_0805, up5k-synth:CP_EIA-2012-15_AVX-P_Pad1.30x1.05mm_HandSolder, F.Cu at (36.0, 4.00)
- added C26: CP_10uF_10v_0805, up5k-synth:CP_EIA-2012-15_AVX-P_Pad1.30x1.05mm_HandSolder, F.Cu at (40.9, 4.00)
- added C27: CP_270uF_10v_PXF, up5k-synth:CP_Elec_6.3x5.8, F.Cu at (38.8, -9.63)
- added C28: CP_270uF_10v_PXF, up5k-synth:CP_Elec_6.3x5.8, F.Cu at (38.8, -1.48)
- added C29: CP_10uF_10v_0805, up5k-synth:CP_EIA-2012-15_AVX-P_Pad1.30x1.05mm_HandSolder, F.Cu at (36.0, 6.81)
- added C30: CP_10uF_10v_0805, up5k-synth:CP_EIA-2012-15_AVX-P_Pad1.30x1.05mm_HandSolder, F.Cu at (40.9, 6.81)
- added C31: 0.1uF_10V_0603, up5k-synth:C_0603_1608Metric_Pad1.08x0.95mm_HandSolder, F.Cu at (56.6, 3.56)
- added C32: CP_10uF_10v_0805, up5k-synth:CP_EIA-2012-15_AVX-P_Pad1.30x1.05mm_HandSolder, F.Cu at (45.7, 4.00)
- added C33: CP_10uF_10v_0805, up5k-synth:CP_EIA-2012-15_AVX-P_Pad1.30x1.05mm_HandSolder, F.Cu at (67.8, -12.3)
- added C34: CP_270uF_10v_PXF, up5k-synth:CP_Elec_6.3x5.8, F.Cu at (49.2, -9.63)
- added C35: CP_10uF_10v_0805, up5k-synth:CP_EIA-2012-15_AVX-P_Pad1.30x1.05mm_HandSolder, F.Cu at (50.5, 4.00)
- added C36: CP_270uF_10v_PXF, up5k-synth:CP_Elec_6.3x5.8, F.Cu at (49.2, -1.48)
- added C37: CP_10uF_10v_0805, up5k-synth:CP_EIA-2012-15_AVX-P_Pad1.30x1.05mm_HandSolder, F.Cu at (45.7, 6.81)
- added C38: 0.1uF_10V_0603, up5k-synth:C_0603_1608Metric_Pad1.08x0.95mm_HandSolder, F.Cu at (56.6, 1.05)
- added R51: R_50kR_4xArray_1206, up5k-synth:R_Array_Convex_4x1206, F.Cu at (62.6, -3.58)
- added R52: R_50kR_4xArray_1206, up5k-synth:R_Array_Convex_4x1206, F.Cu at (57.2, -3.58)
- added R53: R_16R_0603, up5k-synth:R_0603_1608Metric_Pad0.98x0.95mm_HandSolder, F.Cu at (50.3, 6.66)
- added R54: R_16R_0603, up5k-synth:R_0603_1608Metric_Pad0.98x0.95mm_HandSolder, F.Cu at (61.0, 1.05)
- added R55: R_50kR_0603, up5k-synth:R_0603_1608Metric_Pad0.98x0.95mm_HandSolder, F.Cu at (54.6, 6.66)
- added R56: R_50kR_0603, up5k-synth:R_0603_1608Metric_Pad0.98x0.95mm_HandSolder, F.Cu at (67.5, -9.64)
- added R57: R_50kR_4xArray_1206, up5k-synth:R_Array_Convex_4x1206, F.Cu at (62.6, -10.3)
- added R58: R_50kR_4xArray_1206, up5k-synth:R_Array_Convex_4x1206, F.Cu at (57.2, -10.3)
- added R59: R_16R_0603, up5k-synth:R_0603_1608Metric_Pad0.98x0.95mm_HandSolder, F.Cu at (67.5, -7.13)
- added R60: R_16R_0603, up5k-synth:R_0603_1608Metric_Pad0.98x0.95mm_HandSolder, F.Cu at (61.0, 3.56)
- added R61: R_50kR_0603, up5k-synth:R_0603_1608Metric_Pad0.98x0.95mm_HandSolder, F.Cu at (67.5, -4.62)
- added R62: R_50kR_0603, up5k-synth:R_0603_1608Metric_Pad0.98x0.95mm_HandSolder, F.Cu at (65.3, 1.05)
Connections:
- J5 pad 1: Net-(J5-Pad1) -> GND
- J5 pad 2: Net-(J5-Pad2) -> /OUT0_R
- J5 pad 5: Net-(J5-Pad5) -> /OUT0_L
- J6 pad 1: Net-(J6-Pad1) -> GND
- J6 pad 2: Net-(J6-Pad2) -> /OUT1_R
- J6 pad 5: Net-(J6-Pad5) -> /OUT1_L
- U10 pad 1: Net-(U10-Pad1) -> Net-(R53-Pad1)
- U10 pad 2: Net-(U10-Pad2) -> Net-(R53-Pad1)
- U10 pad 4: Net-(U10-Pad4) -> GND
- U10 pad 6: Net-(U10-Pad6) -> Net-(R54-Pad1)
- U10 pad 7: Net-(U10-Pad7) -> Net-(R54-Pad1)
- U10 pad 8: Net-(U10-Pad8) -> +3V3
- U11 pad 1: Net-(U11-Pad1) -> Net-(R59-Pad1)
- U11 pad 2: Net-(U11-Pad2) -> Net-(R59-Pad1)
- U11 pad 4: Net-(U11-Pad4) -> GND
- U11 pad 6: Net-(U11-Pad6) -> Net-(R60-Pad1)
- U11 pad 7: Net-(U11-Pad7) -> Net-(R60-Pad1)
- U11 pad 8: Net-(U11-Pad8) -> +3V3
- U3 pad 11: Net-(U3-Pad11) -> /BUF1_R
- U3 pad 6: Net-(U3-Pad6) -> /BUF1_L
- U9 pad 11: Net-(U9-Pad11) -> /BUF0_R
- U9 pad 6: Net-(U9-Pad6) -> /BUF0_L

Commit message: WIP
Parts:
- added D10: WS2812B, up5k-synth:LED_WS2812B_PLCC4_5.0x5.0mm_P3.2mm, F.Cu at (171.8, -20.5)
- added D11: WS2812B, up5k-synth:LED_WS2812B_PLCC4_5.0x5.0mm_P3.2mm, F.Cu at (155.0, -0.64)
- added D12: WS2812B, up5k-synth:LED_WS2812B_PLCC4_5.0x5.0mm_P3.2mm, F.Cu at (163.4, -7.26)
- added D13: WS2812B, up5k-synth:LED_WS2812B_PLCC4_5.0x5.0mm_P3.2mm, F.Cu at (171.8, -13.9)
- added D14: WS2812B, up5k-synth:LED_WS2812B_PLCC4_5.0x5.0mm_P3.2mm, F.Cu at (180.3, -20.5)
- added D15: WS2812B, up5k-synth:LED_WS2812B_PLCC4_5.0x5.0mm_P3.2mm, F.Cu at (163.4, -0.64)
- added D16: WS2812B, up5k-synth:LED_WS2812B_PLCC4_5.0x5.0mm_P3.2mm, F.Cu at (171.8, -7.26)
- added D17: WS2812B, up5k-synth:LED_WS2812B_PLCC4_5.0x5.0mm_P3.2mm, F.Cu at (180.3, -13.9)
- added D18: WS2812B, up5k-synth:LED_WS2812B_PLCC4_5.0x5.0mm_P3.2mm, F.Cu at (188.7, -20.5)
- added D19: WS2812B, up5k-synth:LED_WS2812B_PLCC4_5.0x5.0mm_P3.2mm, F.Cu at (171.8, -0.64)
- added D20: WS2812B, up5k-synth:LED_WS2812B_PLCC4_5.0x5.0mm_P3.2mm, F.Cu at (180.3, -7.26)
- added D5: WS2812B, up5k-synth:LED_WS2812B_PLCC4_5.0x5.0mm_P3.2mm, F.Cu at (155.0, -20.5)
- added D6: WS2812B, up5k-synth:LED_WS2812B_PLCC4_5.0x5.0mm_P3.2mm, F.Cu at (155.0, -13.9)
- added D7: WS2812B, up5k-synth:LED_WS2812B_PLCC4_5.0x5.0mm_P3.2mm, F.Cu at (163.4, -20.5)
- added D8: WS2812B, up5k-synth:LED_WS2812B_PLCC4_5.0x5.0mm_P3.2mm, F.Cu at (155.0, -7.26)
- added D9: WS2812B, up5k-synth:LED_WS2812B_PLCC4_5.0x5.0mm_P3.2mm, F.Cu at (163.4, -13.9)
- added R51: R_20mR_0603, up5k-synth:R_0603_1608Metric_Pad0.98x0.95mm_HandSolder, F.Cu at (195.1, -22.6)
- added U12: DS2745, up5k-synth:TSSOP-8_3x3mm_P0.65mm, F.Cu at (187.9, -14.9)
Connections:
- B1 pad 2: GND -> -BATT
- U1 pad 89: /mcu_core -> Net-(C7-Pad1)
- U10 pad 3: Net-(C25-Pad1) -> /BUF0_L
- U10 pad 5: Net-(C26-Pad1) -> /BUF0_R
- U11 pad 3: Net-(C32-Pad1) -> /BUF1_L
- U11 pad 5: Net-(C33-Pad1) -> /BUF1_R

Commit message: Design checkpoint at 20210617
Parts:
- added C25: 0.1uF_10V_0603, up5k-synth:C_0603_1608Metric_Pad1.08x0.95mm_HandSolder, F.Cu at (105.5, 100.5)
- added C26: 0.1uF_10V_0603, up5k-synth:C_0603_1608Metric_Pad1.08x0.95mm_HandSolder, F.Cu at (128.2, 113.9)
- added C29: 0.1uF_10V_0603, up5k-synth:C_0603_1608Metric_Pad1.08x0.95mm_HandSolder, F.Cu at (136.9, 112.6)
- added C30: 0.1uF_10V_0603, up5k-synth:C_0603_1608Metric_Pad1.08x0.95mm_HandSolder, F.Cu at (128.7, 119.8)
- added C32: 0.1uF_10V_0603, up5k-synth:C_0603_1608Metric_Pad1.08x0.95mm_HandSolder, F.Cu at (141.7, 107.6)
- added C33: 0.1uF_10V_0603, up5k-synth:C_0603_1608Metric_Pad1.08x0.95mm_HandSolder, F.Cu at (131.0, 116.4)
- added C35: 0.1uF_10V_0603, up5k-synth:C_0603_1608Metric_Pad1.08x0.95mm_HandSolder, F.Cu at (141.7, 105.1)
- added C37: 0.1uF_10V_0603, up5k-synth:C_0603_1608Metric_Pad1.08x0.95mm_HandSolder, F.Cu at (137.3, 110.1)
- added C39: 0.1uF_10V_0603, up5k-synth:C_0603_1608Metric_Pad1.08x0.95mm_HandSolder, F.Cu at (132.6, 113.5)
- added C40: 0.1uF_10V_0603, up5k-synth:C_0603_1608Metric_Pad1.08x0.95mm_HandSolder, F.Cu at (124.3, 119.9)
- added C41: 0.1uF_10V_0603, up5k-synth:C_0603_1608Metric_Pad1.08x0.95mm_HandSolder, F.Cu at (137.3, 107.6)
- added C42: 0.1uF_10V_0603, up5k-synth:C_0603_1608Metric_Pad1.08x0.95mm_HandSolder, F.Cu at (126.7, 117.3)
- added C43: 0.1uF_10V_0603, up5k-synth:C_0603_1608Metric_Pad1.08x0.95mm_HandSolder, F.Cu at (132.6, 111.0)
- added C44: 0.1uF_10V_0603, up5k-synth:C_0603_1608Metric_Pad1.08x0.95mm_HandSolder, F.Cu at (137.3, 105.1)
- added C45: 0.1uF_10V_0603, up5k-synth:C_0603_1608Metric_Pad1.08x0.95mm_HandSolder, F.Cu at (140.9, 102.6)
- added C46: 0.1uF_10V_0603, up5k-synth:C_0603_1608Metric_Pad1.08x0.95mm_HandSolder, F.Cu at (132.9, 108.5)
- added C47: 0.1uF_10V_0603, up5k-synth:C_0603_1608Metric_Pad1.08x0.95mm_HandSolder, F.Cu at (105.5, 103.0)
- added C48: 0.1uF_10V_0603, up5k-synth:C_0603_1608Metric_Pad1.08x0.95mm_HandSolder, F.Cu at (120.0, 119.9)
- added C49: 0.1uF_10V_0603, up5k-synth:C_0603_1608Metric_Pad1.08x0.95mm_HandSolder, F.Cu at (140.9, 100.0)
- added C50: 0.1uF_10V_0603, up5k-synth:C_0603_1608Metric_Pad1.08x0.95mm_HandSolder, F.Cu at (122.3, 117.4)
- added C51: 0.1uF_10V_0603, up5k-synth:C_0603_1608Metric_Pad1.08x0.95mm_HandSolder, F.Cu at (128.2, 111.4)
- added C52: 0.1uF_10V_0603, up5k-synth:C_0603_1608Metric_Pad1.08x0.95mm_HandSolder, F.Cu at (132.9, 106.0)
- added C53: 0.1uF_10V_0603, up5k-synth:C_0603_1608Metric_Pad1.08x0.95mm_HandSolder, F.Cu at (136.6, 102.6)
- added C54: 0.1uF_10V_0603, up5k-synth:C_0603_1608Metric_Pad1.08x0.95mm_HandSolder, F.Cu at (128.2, 108.9)
- added C55: 0.1uF_10V_0603, up5k-synth:C_0603_1608Metric_Pad1.08x0.95mm_HandSolder, F.Cu at (123.5, 114.8)
- added C56: 0.1uF_10V_0603, up5k-synth:C_0603_1608Metric_Pad1.08x0.95mm_HandSolder, F.Cu at (141.3, 97.1)
- added C57: 0.1uF_10V_0603, up5k-synth:C_0603_1608Metric_Pad1.08x0.95mm_HandSolder, F.Cu at (115.7, 120.3)
- added C58: 0.1uF_10V_0603, up5k-synth:C_0603_1608Metric_Pad1.08x0.95mm_HandSolder, F.Cu at (136.6, 100.0)
- added C59: 0.1uF_10V_0603, up5k-synth:C_0603_1608Metric_Pad1.08x0.95mm_HandSolder, F.Cu at (118.0, 117.4)
- added C60: 0.1uF_10V_0603, up5k-synth:C_0603_1608Metric_Pad1.08x0.95mm_HandSolder, F.Cu at (111.3, 120.3)
- added R52: 360kR, up5k-synth:R_0805_2012Metric_Pad1.20x1.40mm_HandSolder, F.Cu at (132.0, 94.4)
- added R57: 360kR, up5k-synth:R_0805_2012Metric_Pad1.20x1.40mm_HandSolder, F.Cu at (118.9, 105.8)
- added R58: 360kR, up5k-synth:R_0805_2012Metric_Pad1.20x1.40mm_HandSolder, F.Cu at (136.8, 97.3)
- added R63: 360kR, up5k-synth:R_0805_2012Metric_Pad1.20x1.40mm_HandSolder, F.Cu at (106.8, 120.2)
- added R64: 360kR, up5k-synth:R_0805_2012Metric_Pad1.20x1.40mm_HandSolder, F.Cu at (123.7, 109.1)
- added R65: 360kR, up5k-synth:R_0805_2012Metric_Pad1.20x1.40mm_HandSolder, F.Cu at (118.9, 114.7)
- added R66: 360kR, up5k-synth:R_0805_2012Metric_Pad1.20x1.40mm_HandSolder, F.Cu at (123.7, 112.1)
- added R67: 360kR, up5k-synth:R_0805_2012Metric_Pad1.20x1.40mm_HandSolder, F.Cu at (132.0, 103.2)
- added R68: 360kR, up5k-synth:R_0805_2012Metric_Pad1.20x1.40mm_HandSolder, F.Cu at (141.5, 94.4)
- added R69: 360kR, up5k-synth:R_0805_2012Metric_Pad1.20x1.40mm_HandSolder, F.Cu at (132.0, 100.3)
- added R70: 360kR, up5k-synth:R_0805_2012Metric_Pad1.20x1.40mm_HandSolder, F.Cu at (118.9, 108.8)
- added R71: 360kR, up5k-synth:R_0805_2012Metric_Pad1.20x1.40mm_HandSolder, F.Cu at (113.4, 117.6)
- added R72: 360kR, up5k-synth:R_0805_2012Metric_Pad1.20x1.40mm_HandSolder, F.Cu at (123.7, 106.2)
- added R73: 360kR, up5k-synth:R_0805_2012Metric_Pad1.20x1.40mm_HandSolder, F.Cu at (136.8, 94.4)
- added R74: 360kR, up5k-synth:R_0805_2012Metric_Pad1.20x1.40mm_HandSolder, F.Cu at (118.9, 111.7)
- added R75: 360kR, up5k-synth:R_0805_2012Metric_Pad1.20x1.40mm_HandSolder, F.Cu at (127.3, 103.2)
- added R76: 360kR, up5k-synth:R_0805_2012Metric_Pad1.20x1.40mm_HandSolder, F.Cu at (114.2, 114.7)
- added R77: 360kR, up5k-synth:R_0805_2012Metric_Pad1.20x1.40mm_HandSolder, F.Cu at (132.0, 97.3)
- added R78: 360kR, up5k-synth:R_0805_2012Metric_Pad1.20x1.40mm_HandSolder, F.Cu at (127.3, 100.3)
- added R79: 360kR, up5k-synth:R_0805_2012Metric_Pad1.20x1.40mm_HandSolder, F.Cu at (128.4, 106.2)
- added R80: 360kR, up5k-synth:R_0805_2012Metric_Pad1.20x1.40mm_HandSolder, F.Cu at (97.2, 118.4)
- added R81: 360kR, up5k-synth:R_0805_2012Metric_Pad1.20x1.40mm_HandSolder, F.Cu at (127.3, 94.4)
- added R82: 360kR, up5k-synth:R_0805_2012Metric_Pad1.20x1.40mm_HandSolder, F.Cu at (114.2, 105.8)
- added R83: 360kR, up5k-synth:R_0805_2012Metric_Pad1.20x1.40mm_HandSolder, F.Cu at (114.2, 108.8)
- added R84: 360kR, up5k-synth:R_0805_2012Metric_Pad1.20x1.40mm_HandSolder, F.Cu at (127.3, 97.3)
- added R85: 360kR, up5k-synth:R_0805_2012Metric_Pad1.20x1.40mm_HandSolder, F.Cu at (102.0, 120.2)
- added R86: 360kR, up5k-synth:R_0805_2012Metric_Pad1.20x1.40mm_HandSolder, F.Cu at (108.7, 117.3)
- added R87: 360kR, up5k-synth:R_0805_2012Metric_Pad1.20x1.40mm_HandSolder, F.Cu at (114.2, 111.7)
- added R88: 360kR, up5k-synth:R_0805_2012Metric_Pad1.20x1.40mm_HandSolder, F.Cu at (103.9, 117.3)
- added SW26: SW_DPDT_x2_MFS201N−16−Z, up5k-synth:SW_E-Switch_MFS201N−16−Z_DPDT, F.Cu at (97.6, 94.5)
- added U13: DSC6003JI2A, up5k-synth:Oscillator_SMD_TXC_7C-4Pin_5.0x3.2mm_HandSoldering, F.Cu at (98.2, 113.8)
- added U14: 74HC165, up5k-synth:SO-16_3.9x9.9mm_P1.27mm, F.Cu at (120.7, 98.6)
- added U15: 74HC165, up5k-synth:SO-16_3.9x9.9mm_P1.27mm, F.Cu at (107.5, 110.1)
- added U16: 74HC165, up5k-synth:SO-16_3.9x9.9mm_P1.27mm, F.Cu at (112.2, 98.6)
- added U17: 74HC165, up5k-synth:SO-16_3.9x9.9mm_P1.27mm, F.Cu at (99.1, 105.0)
Connections:
- ENC1 pad 1: Net-(ENC1-Pad1) -> +3V3
- ENC1 pad 2: Net-(ENC1-Pad2) -> /SW_ENC1
- ENC1 pad 3: Net-(ENC1-Pad3) -> /ENC1_A
- ENC1 pad 4: Net-(ENC1-Pad4) -> +3V3
- ENC1 pad 5: Net-(ENC1-Pad5) -> /ENC1_B
- ENC2 pad 1: Net-(ENC2-Pad1) -> +3V3
- ENC2 pad 2: Net-(ENC2-Pad2) -> /SW_ENC2
- ENC2 pad 3: Net-(ENC2-Pad3) -> /ENC2_A
- ENC2 pad 4: Net-(ENC2-Pad4) -> +3V3
- ENC2 pad 5: Net-(ENC2-Pad5) -> /ENC2_B
- R3 pad 2: /Vout -> /PSU_EN
- U1 pad 21: Net-(U1-Pad21) -> /SW_DATA
- U1 pad 22: Net-(U1-Pad22) -> /SW_CLK
- U1 pad 23: Net-(U1-Pad23) -> /SW_LOAD
- U1 pad 48: /MII_GTXCK -> /MII_GRXCK
- U1 pad 89: Net-(C7-Pad1) -> /mcu_core
- U2 pad 24: Net-(U2-Pad24) -> +3V3
- U2 pad 29: Net-(U2-Pad29) -> +1V2
- U2 pad 6: /MII_GRDV -> Net-(U2-Pad6)
- U4 pad 5: /Vout -> /PSU_EN
