File: synth/synth.kicad_pcb (KiCad board)
At the start: 2 copper layers, 210 parts, among them J1 MEM2061-01-188-00-A, J2 10118194-0001LF, J3 PMOD_conn, J5 AudioJack3_SwitchTR, J6 AudioJack3_SwitchTR, SW26 SW_DPDT_x2_MFS201N−16−Z, U1 ATSAME53N19A, U10 AD8531, U11 AD8531, U12 DS2745, U13 DSC6003JI2A, U14 74HC165, U15 74HC165, U16 74HC165, U17 74HC165, U2 DRA818_iCE40-UP5K-SG48, U3 DS1881, U4 LMS33460, U5 TPS62120DCNR, U6 BQ24074, U7 DSC6003JI2A, U8 TPS63031, U9 DS1881

Commit message: Design checkpoint at 20210617
Parts:
- added C61: C_150pF_10V_0603, up5k-synth:C_0603_1608Metric_Pad1.08x0.95mm_HandSolder, F.Cu at (126.0, 18.0)
- added C62: C_150pF_10V_0603, up5k-synth:C_0603_1608Metric_Pad1.08x0.95mm_HandSolder, F.Cu at (126.0, 20.5)
- added C63: C_150pF_10V_0603, up5k-synth:C_0603_1608Metric_Pad1.08x0.95mm_HandSolder, F.Cu at (130.3, 18.0)
- added C64: C_150pF_10V_0603, up5k-synth:C_0603_1608Metric_Pad1.08x0.95mm_HandSolder, F.Cu at (126.0, 23.0)
- added P1: keypad, up5k-synth:DIY_KEYPAD, F.Cu at (32.0, 94.0)
- added P10: keypad, up5k-synth:DIY_KEYPAD, F.Cu at (131.0, 94.0)
- added P11: keypad, up5k-synth:DIY_KEYPAD, F.Cu at (142.0, 94.0)
- added P12: keypad, up5k-synth:DIY_KEYPAD, F.Cu at (-50.3, 89.1)
- added P13: keypad, up5k-synth:DIY_KEYPAD, F.Cu at (-32.5, 75.5)
- added P14: keypad, up5k-synth:DIY_KEYPAD, F.Cu at (-14.6, 62.0)
- added P15: keypad, up5k-synth:DIY_KEYPAD, F.Cu at (-50.3, 102.7)
- added P16: keypad, up5k-synth:DIY_KEYPAD, F.Cu at (-32.5, 89.1)
- added P17: keypad, up5k-synth:DIY_KEYPAD, F.Cu at (-14.6, 75.5)
- added P18: keypad, up5k-synth:DIY_KEYPAD, F.Cu at (3.25, 62.0)
- added P19: keypad, up5k-synth:DIY_KEYPAD, F.Cu at (-32.5, 102.7)
- added P2: keypad, up5k-synth:DIY_KEYPAD, F.Cu at (43.0, 94.0)
- added P20: keypad, up5k-synth:DIY_KEYPAD, F.Cu at (-14.6, 89.1)
- added P21: keypad, up5k-synth:DIY_KEYPAD, F.Cu at (3.25, 75.5)
- added P22: keypad, up5k-synth:DIY_KEYPAD, F.Cu at (-14.6, 102.7)
- added P23: keypad, up5k-synth:DIY_KEYPAD, F.Cu at (3.25, 89.1)
- added P24: keypad, up5k-synth:DIY_KEYPAD, F.Cu at (3.25, 102.7)
- added P3: keypad, up5k-synth:DIY_KEYPAD, F.Cu at (54.0, 94.0)
- added P4: keypad, up5k-synth:DIY_KEYPAD, F.Cu at (65.0, 94.0)
- added P5: keypad, up5k-synth:DIY_KEYPAD, F.Cu at (76.0, 94.0)
- added P6: keypad, up5k-synth:DIY_KEYPAD, F.Cu at (87.0, 94.0)
- added P7: keypad, up5k-synth:DIY_KEYPAD, F.Cu at (98.0, 94.0)
- added P8: keypad, up5k-synth:DIY_KEYPAD, F.Cu at (109.0, 94.0)
- added P9: keypad, up5k-synth:DIY_KEYPAD, F.Cu at (120.0, 94.0)
- added R89: R_36kR_0603, up5k-synth:R_0603_1608Metric_Pad0.98x0.95mm_HandSolder, F.Cu at (130.3, 20.5)
- added R90: R_36kR_0603, up5k-synth:R_0603_1608Metric_Pad0.98x0.95mm_HandSolder, F.Cu at (134.7, 18.0)
- added R91: R_36kR_0603, up5k-synth:R_0603_1608Metric_Pad0.98x0.95mm_HandSolder, F.Cu at (130.3, 23.0)
- added R92: R_36kR_0603, up5k-synth:R_0603_1608Metric_Pad0.98x0.95mm_HandSolder, F.Cu at (134.7, 20.5)
- added SW1: SW_Push, up5k-synth:SW_Push_1P1T_NO_6x6mm_H9.5mm, B.Cu at (34.0, 31.0)
- added SW10: SW_Push, up5k-synth:SW_Push_1P1T_NO_6x6mm_H9.5mm, F.Cu at (108.8, 75.9)
- added SW11: SW_Push, up5k-synth:SW_Push_1P1T_NO_6x6mm_H9.5mm, F.Cu at (126.3, 62.1)
- added SW12: SW_Push, up5k-synth:SW_Push_1P1T_NO_6x6mm_H9.5mm, F.Cu at (51.1, 75.5)
- added SW13: SW_Push, up5k-synth:SW_Push_1P1T_NO_6x6mm_H9.5mm, F.Cu at (62.0, 76.0)
- added SW14: SW_Push, up5k-synth:SW_Push_1P1T_NO_6x6mm_H9.5mm, F.Cu at (37.3, 34.9)
- added SW15: SW_Push, up5k-synth:SW_Push_1P1T_NO_6x6mm_H9.5mm, F.Cu at (126.7, 75.9)
- added SW16: SW_Push, up5k-synth:SW_Push_1P1T_NO_6x6mm_H9.5mm, F.Cu at (144.2, 62.1)
- added SW17: SW_Push, up5k-synth:SW_Push_1P1T_NO_6x6mm_H9.5mm, F.Cu at (73.0, 75.5)
- added SW18: SW_Push, up5k-synth:SW_Push_1P1T_NO_6x6mm_H9.5mm, F.Cu at (90.8, 62.0)
- added SW19: SW_Push, up5k-synth:SW_Push_1P1T_NO_6x6mm_H9.5mm, F.Cu at (74.0, 65.0)
- added SW2: SW_Push, up5k-synth:SW_Push_1P1T_NO_6x6mm_H9.5mm, F.Cu at (37.3, 48.5)
- added SW20: SW_Push, up5k-synth:SW_Push_1P1T_NO_6x6mm_H9.5mm, F.Cu at (144.6, 75.9)
- added SW21: SW_Push, up5k-synth:SW_Push_1P1T_NO_6x6mm_H9.5mm, F.Cu at (162.0, 62.1)
- added SW22: SW_Push, up5k-synth:SW_Push_1P1T_NO_6x6mm_H9.5mm, F.Cu at (90.8, 75.5)
- added SW23: SW_Push, up5k-synth:SW_Push_1P1T_NO_6x6mm_H9.5mm, F.Cu at (108.7, 62.0)
- added SW24: SW_Push, up5k-synth:SW_Push_1P1T_NO_6x6mm_H9.5mm, F.Cu at (77.0, 55.0)
- added SW25: SW_Push, up5k-synth:SW_Push_1P1T_NO_6x6mm_H9.5mm, F.Cu at (160.0, 75.0)
- added SW3: SW_Push, up5k-synth:SW_Push_1P1T_NO_6x6mm_H9.5mm, F.Cu at (51.1, 34.9)
- added SW4: SW_Push, up5k-synth:SW_Push_1P1T_NO_6x6mm_H9.5mm, F.Cu at (37.3, 62.0)
- added SW5: SW_Push, up5k-synth:SW_Push_1P1T_NO_6x6mm_H9.5mm, F.Cu at (51.1, 48.5)
- added SW6: SW_Push, up5k-synth:SW_Push_1P1T_NO_6x6mm_H9.5mm, F.Cu at (62.0, 34.9)
- added SW7: SW_Push, up5k-synth:SW_Push_1P1T_NO_6x6mm_H9.5mm, F.Cu at (37.3, 75.5)
- added SW8: SW_Push, up5k-synth:SW_Push_1P1T_NO_6x6mm_H9.5mm, F.Cu at (51.1, 62.0)
- added SW9: SW_Push, up5k-synth:SW_Push_1P1T_NO_6x6mm_H9.5mm, F.Cu at (63.0, 48.0)
- U12: moved to B.Cu
- moved ENC1 125.7 mm to (-25.5, -43.5)
- moved ENC2 125.7 mm to (-43.5, -32.5)
- moved J3 125.7 mm to (-33.5, -58.5)
- moved J5 125.7 mm to (-45.5, -47.5)
- moved R36 101.9 mm to (122.5, 155.8)
- moved R41 101.9 mm to (127.2, 155.8)
- moved R46 101.9 mm to (132.0, 155.8)
- moved R49 101.9 mm to (136.8, 155.8)
- moved C7 101.9 mm to (152.5, 160.5)
- moved R1 101.9 mm to (147.0, 162.5)
- moved R2 101.9 mm to (147.0, 157.5)
- moved R27 101.9 mm to (122.5, 144.0)
- moved R29 101.9 mm to (127.2, 144.0)
- moved R30 101.9 mm to (122.5, 149.9)
- moved R32 101.9 mm to (132.0, 144.0)
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Connections:
- D10 pad 1: Net-(D10-Pad1) -> +3V3
- D10 pad 3: Net-(D10-Pad3) -> GND
- D11 pad 1: Net-(D11-Pad1) -> +3V3
- D11 pad 3: Net-(D11-Pad3) -> GND
- D11 pad 4: Net-(D11-Pad4) -> Net-(D10-Pad2)
- D12 pad 1: Net-(D12-Pad1) -> +3V3
- D12 pad 2: Net-(D12-Pad2) -> /LED_DOUT
- D12 pad 3: Net-(D12-Pad3) -> GND
- D12 pad 4: Net-(D12-Pad4) -> Net-(D11-Pad2)
- D13 pad 1: Net-(D13-Pad1) -> +3V3
- D13 pad 3: Net-(D13-Pad3) -> GND
- D13 pad 4: Net-(D13-Pad4) -> /LED_DOUT
- D14 pad 1: Net-(D14-Pad1) -> +3V3
- D14 pad 3: Net-(D14-Pad3) -> GND
- D14 pad 4: Net-(D14-Pad4) -> Net-(D13-Pad2)
- D15 pad 1: Net-(D15-Pad1) -> +3V3
- D15 pad 3: Net-(D15-Pad3) -> GND
- D15 pad 4: Net-(D15-Pad4) -> Net-(D14-Pad2)
- D16 pad 1: Net-(D16-Pad1) -> +3V3
- D16 pad 3: Net-(D16-Pad3) -> GND
- D16 pad 4: Net-(D16-Pad4) -> Net-(D15-Pad2)
- D17 pad 1: Net-(D17-Pad1) -> +3V3
- D17 pad 3: Net-(D17-Pad3) -> GND
- D17 pad 4: Net-(D17-Pad4) -> Net-(D16-Pad2)
- D18 pad 1: Net-(D18-Pad1) -> +3V3
- D18 pad 3: Net-(D18-Pad3) -> GND
- D18 pad 4: Net-(D18-Pad4) -> Net-(D17-Pad2)
- D19 pad 1: Net-(D19-Pad1) -> +3V3
- D19 pad 3: Net-(D19-Pad3) -> GND
- D19 pad 4: Net-(D19-Pad4) -> Net-(D18-Pad2)
- D20 pad 1: Net-(D20-Pad1) -> +3V3
- D20 pad 3: Net-(D20-Pad3) -> GND
- D20 pad 4: Net-(D20-Pad4) -> Net-(D19-Pad2)
- D5 pad 1: Net-(D5-Pad1) -> +3V3
- D5 pad 3: Net-(D5-Pad3) -> GND
- D5 pad 4: Net-(D5-Pad4) -> /LED_DATA
- D6 pad 1: Net-(D6-Pad1) -> +3V3
- D6 pad 3: Net-(D6-Pad3) -> GND
- D6 pad 4: Net-(D6-Pad4) -> Net-(D5-Pad2)
- D7 pad 1: Net-(D7-Pad1) -> +3V3
- D7 pad 3: Net-(D7-Pad3) -> GND
- D7 pad 4: Net-(D7-Pad4) -> Net-(D6-Pad2)
- D8 pad 1: Net-(D8-Pad1) -> +3V3
- D8 pad 3: Net-(D8-Pad3) -> GND
- D8 pad 4: Net-(D8-Pad4) -> Net-(D7-Pad2)
- D9 pad 1: Net-(D9-Pad1) -> +3V3
- D9 pad 2: Net-(D9-Pad2) -> Net-(D10-Pad4)
- D9 pad 3: Net-(D9-Pad3) -> GND
- D9 pad 4: Net-(D9-Pad4) -> Net-(D8-Pad2)
- U1 pad 96: Net-(U1-Pad96) -> /LED_DATA
- U3 pad 10: /PDM1_R -> /F_PDM1_R
- U3 pad 8: /PDM1_L -> /F_PDM1_L
- U9 pad 10: /PDM0_R -> /F_PDM0_R
- U9 pad 8: /PDM0_L -> /F_PDM0_L

Commit message: Design checkpoint at 20210621
Parts:
- removed the R51 at (62.6, -3.58)
- removed the R52 at (82.0, 153.4)
- removed the R52 at (57.2, -3.58)
- removed the R57 at (68.9, 164.8)
- removed the R57 at (62.6, -10.3)
- removed the R58 at (86.8, 156.3)
- removed the R58 at (57.2, -10.3)
- added J4: debug_conn, up5k-synth:PinHeader_2x03_P2.54mm_Vertical, B.Cu at (246.7, 86.2)
- added R52: 360kR, up5k-synth:R_0805_2012Metric_Pad1.20x1.40mm_HandSolder, B.Cu at (67.0, 193.6)
- added R57: 360kR, up5k-synth:R_0805_2012Metric_Pad1.20x1.40mm_HandSolder, B.Cu at (53.9, 182.2)
- added R58: 360kR, up5k-synth:R_0805_2012Metric_Pad1.20x1.40mm_HandSolder, B.Cu at (71.8, 190.7)
- added R93: 360kR, up5k-synth:R_0805_2012Metric_Pad1.20x1.40mm_HandSolder, B.Cu at (46.1, 39.4)
- added R94: 360kR, up5k-synth:R_0805_2012Metric_Pad1.20x1.40mm_HandSolder, B.Cu at (46.6, 62.2)
- C1, C10, C11, C12, C13, C14, C15, C16, C17, C18, C19, C2 (x2), C20, C21, C22, C23, C24, C25 (x2), C26 (x2), C27, C28, C29 (x2), C3, C30 (x2), C31, C32 (x2), C33 (x2), C34, C35 (x2), C36, C37 (x2), C38, C39, C4 (x2), C40, C41, C42, C43, C44, C45, C46, C47, C48, C49, C5, C50, C51, C52, C53, C54, C55, C56, C57, C58, C59, C6, C60, C61, C62, C63, C64, C7, C8, C9, D3, D4, J1, J2, L1, L2, R1, R10, R11, R12, R13, R15, R16, R17, R18, R19, R2, R20, R21, R22, R23, R24, R25, R26, R27, R28, R29, R3, R30, R31, R32, R33, R34, R35, R36, R37, R38, R39, R4, R40, R41, R42, R43, R44, R45, R46, R47, R48, R49, R5, R50, R51, R53, R54, R55, R56, R59, R6, R60, R61, R62, R63, R64, R65, R66, R67, R68, R69, R7, R70, R71, R72, R73, R74, R75, R76, R77, R78, R79, R8, R80, R81, R82, R83, R84, R85, R86, R87, R88, R89, R9, R90, R91, R92, U1, U10, U11, U13, U14, U15, U16, U17, U2, U3, U4, U5, U6, U7, U8, U9: moved to B.Cu
- moved J5 345.4 mm to (271.7, 89.2), turned to 270 degrees
- moved D1 252.6 mm to (46.0, 31.0), turned to 90 degrees
- moved P12 251.5 mm to (200.0, 114.0)
- moved C27 250.4 mm to (256.4, 114.2), turned to 180 degrees
- moved D2 246.3 mm to (53.0, 31.0), turned to 90 degrees
- moved J3 241.9 mm to (188.3, 38.0)
- moved C28 238.7 mm to (259.2, 90.0), turned to 270 degrees
- moved J6 233.8 mm to (271.7, 108.2), turned to 270 degrees
- moved C36 233.4 mm to (259.2, 100.4), turned to 270 degrees
- moved C34 229.9 mm to (251.1, 100.4), turned to 270 degrees
- moved P24 200.8 mm to (204.0, 102.0)
- moved P22 194.6 mm to (180.0, 102.0)
- moved P23 189.2 mm to (192.0, 102.0)
- moved P19 176.5 mm to (144.0, 102.0)
- moved P20 171.1 mm to (156.0, 102.0)
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Connections:
- P1 pad 2: Net-(P1-Pad2) -> /ADC0IN[0]
- P10 pad 2: Net-(P10-Pad2) -> /ADC1IN[6]
- P11 pad 2: Net-(P11-Pad2) -> /ADC0IN[7]
- P12 pad 2: Net-(P12-Pad2) -> /ADC1IN[7]
- P13 pad 2: Net-(P13-Pad2) -> /ADC0IN[8]
- P14 pad 2: Net-(P14-Pad2) -> /ADC1IN[8]
- P15 pad 2: Net-(P15-Pad2) -> /ADC0IN[9]
- P16 pad 2: Net-(P16-Pad2) -> /ADC1IN[9]
- P17 pad 2: Net-(P17-Pad2) -> /ADC0IN[10]
- P18 pad 2: Net-(P18-Pad2) -> /ADC0IN[2]
- P19 pad 2: Net-(P19-Pad2) -> /ADC0IN[11]
- P2 pad 2: Net-(P2-Pad2) -> /ADC0IN[12]
- P20 pad 2: Net-(P20-Pad2) -> /ADC0IN[3]
- P21 pad 2: Net-(P21-Pad2) -> /ADC1IN[10]
- P22 pad 2: Net-(P22-Pad2) -> /ADC1IN[4]
- P23 pad 2: Net-(P23-Pad2) -> /ADC1IN[11]
- P24 pad 2: Net-(P24-Pad2) -> /ADC1IN[5]
- P3 pad 2: Net-(P3-Pad2) -> /ADC0IN[1]
- P4 pad 2: Net-(P4-Pad2) -> /ADC0IN[13]
- P5 pad 2: Net-(P5-Pad2) -> /ADC0IN[4]
- P6 pad 2: Net-(P6-Pad2) -> /ADC0IN[14]
- P7 pad 2: Net-(P7-Pad2) -> /ADC0IN[5]
- P8 pad 2: Net-(P8-Pad2) -> /ADC0IN[15]
- P9 pad 2: Net-(P9-Pad2) -> /ADC0IN[6]
- R27 pad 2: Net-(R27-Pad2) -> /ADC0IN[0]
- R28 pad 2: Net-(R28-Pad2) -> /ADC0IN[12]
- R29 pad 2: Net-(R29-Pad2) -> /ADC0IN[1]
- R30 pad 2: Net-(R30-Pad2) -> /ADC0IN[13]
- R31 pad 2: Net-(R31-Pad2) -> /ADC0IN[4]
- R32 pad 2: Net-(R32-Pad2) -> /ADC0IN[14]
- R33 pad 2: Net-(R33-Pad2) -> /ADC0IN[5]
- R34 pad 2: Net-(R34-Pad2) -> /ADC0IN[15]
- R35 pad 2: Net-(R35-Pad2) -> /ADC0IN[6]
- R36 pad 2: Net-(R36-Pad2) -> /ADC1IN[6]
- R37 pad 2: Net-(R37-Pad2) -> /ADC0IN[7]
- R38 pad 2: Net-(R38-Pad2) -> /ADC1IN[7]
- R39 pad 2: Net-(R39-Pad2) -> /ADC0IN[8]
- R40 pad 2: Net-(R40-Pad2) -> /ADC1IN[8]
- R41 pad 2: Net-(R41-Pad2) -> /ADC0IN[9]
- R42 pad 2: Net-(R42-Pad2) -> /ADC1IN[9]
- R43 pad 2: Net-(R43-Pad2) -> /ADC0IN[10]
- R44 pad 2: Net-(R44-Pad2) -> /ADC0IN[2]
- R45 pad 2: Net-(R45-Pad2) -> /ADC0IN[11]
- R46 pad 2: Net-(R46-Pad2) -> /ADC0IN[3]
- R47 pad 2: Net-(R47-Pad2) -> /ADC1IN[10]
- R48 pad 2: Net-(R48-Pad2) -> /ADC1IN[4]
- R49 pad 2: Net-(R49-Pad2) -> /ADC1IN[11]
- R50 pad 2: Net-(R50-Pad2) -> /ADC1IN[5]
- U1 pad 89: /mcu_core -> Net-(C7-Pad1)

Commit message: Design checkpoint on 20210622
Parts:
- added DIS1: SSD1306, up5k-synth:SSD1306, F.Cu at (119.5, 56.0)
- moved R3 285.8 mm to (-5.50, 6.00), turned to 90 degrees
- moved U4 276.7 mm to (-0.50, 5.00), turned to 270 degrees
- moved C19 262.1 mm to (6.00, 9.00), turned to 180 degrees
- moved C23 253.4 mm to (9.50, 13.0), turned to 180 degrees
- moved C22 253.3 mm to (10.5, 9.00), turned to 180 degrees
- moved J5 244.7 mm to (28.3, 114.8), turned to 90 degrees
- moved J6 243.7 mm to (28.3, 95.8), turned to 90 degrees
- moved U8 243.0 mm to (15.1, 12.0), turned to 180 degrees
- moved J1 234.2 mm to (33.5, 57.5), turned to 90 degrees
- moved L2 233.3 mm to (21.5, 7.00), turned to 180 degrees
- moved C21 232.2 mm to (20.5, 12.5), turned to 90 degrees
- moved J2 220.3 mm to (51.5, 31.0), turned to 0 degrees
- moved C28 219.8 mm to (40.8, 114.0), turned to 90 degrees
- moved C36 218.5 mm to (40.8, 103.6), turned to 90 degrees
- moved C27 214.2 mm to (43.6, 89.8), turned to 0 degrees
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Connections:
- U1 pad 89: Net-(C7-Pad1) -> /mcu_core
