File: synth/synth.kicad_pcb (KiCad board)
At the start: 2 copper layers, 267 parts, among them J1 MEM2061-01-188-00-A, J2 10118194-0001LF, J3 PMOD_conn, J4 debug_conn, J5 AudioJack3_SwitchTR, J6 AudioJack3_SwitchTR, P1 keypad, P10 keypad, P11 keypad, P12 keypad, P13 keypad, P14 keypad, P15 keypad, P16 keypad, P17 keypad, P18 keypad, P19 keypad, P2 keypad, P20 keypad, P21 keypad, P22 keypad, P23 keypad, P24 keypad, P3 keypad, P4 keypad, P5 keypad, P6 keypad, P7 keypad, P8 keypad, P9 keypad, SW1 SW_Push, SW10 SW_Push, SW11 SW_Push, SW12 SW_Push, SW13 SW_Push, SW14 SW_Push, SW15 SW_Push, SW16 SW_Push, SW17 SW_Push, SW18 SW_Push, SW19 SW_Push, SW2 SW_Push, SW20 SW_Push, SW21 SW_Push, SW22 SW_Push, SW23 SW_Push, SW24 SW_Push, SW25 SW_Push, SW26 SW_DPDT_x2_MFS201N−16−Z, SW3 SW_Push, SW4 SW_Push, SW5 SW_Push, SW6 SW_Push, SW7 SW_Push, SW8 SW_Push, SW9 SW_Push, U1 ATSAME53N19A, U10 AD8531, U11 AD8531, U12 DS2745, U13 DSC6003JI2A, U14 74HC165, U15 74HC165, U16 74HC165, U17 74HC165, U2 DRA818_iCE40-UP5K-SG48, U3 DS1881, U4 LMS33460, U5 TPS62120DCNR, U6 BQ24074, U7 DSC6003JI2A, U8 TPS63031, U9 DS1881

Commit message: Design checkpoint at 20210624
Parts:
- R5, R6: moved to F.Cu
- moved R3 266.2 mm to (243.5, 100.0), turned to 0 degrees
- moved U4 264.6 mm to (244.5, 105.0), turned to 180 degrees
- moved SW26 246.1 mm to (268.5, 96.5)
- moved C21 231.1 mm to (238.0, 90.5)
- moved C22 231.1 mm to (228.0, 87.0)
- moved C23 231.1 mm to (227.0, 91.0)
- moved L2 231.1 mm to (239.0, 85.0)
- moved U8 231.1 mm to (232.6, 90.0)
- moved J2 218.3 mm to (269.0, 49.5), turned to 270 degrees
- moved J1 212.9 mm to (245.0, 33.5), turned to 0 degrees
- moved R4 211.4 mm to (263.5, 52.5), turned to 270 degrees
- moved D4 211.2 mm to (261.0, 50.0), turned to 270 degrees
- moved D3 209.1 mm to (258.5, 49.5), turned to 270 degrees
- moved R15 205.5 mm to (252.0, 46.5), turned to 270 degrees
- moved C14 199.9 mm to (251.4, 51.5), turned to 0 degrees
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
Commit message: Design checkpoint @20210628
Parts:
- removed C19: 4.7uF_10V_0805, up5k-synth:C_0805_2012Metric_Pad1.18x1.45mm_HandSolder
- removed the C2 at (243.5, 79.5)
- removed the C2 at (246.0, 92.5)
- removed C22: 10uF_10V_0805, up5k-synth:C_0805_2012Metric_Pad1.18x1.45mm_HandSolder
- removed the C25 at (40.5, 187.5)
- removed the C25 at (33.0, -5.00)
- removed the C26 at (63.2, 174.1)
- removed the C26 at (37.9, -5.00)
- removed C27, C28: CP_270uF_10v_PXF, up5k-synth:CP_Elec_6.3x5.8
- removed the C29 at (71.9, 175.4)
- removed the C29 at (33.0, -7.81)
- removed C30, C32, C33, C35, C37, C38, C39, C40, C45, C46: 0.1uF_10V_0603, up5k-synth:C_0603_1608Metric_Pad1.08x0.95mm_HandSolder
- removed C30, C32, C33, C35, C37: CP_10uF_10v_0805, up5k-synth:CP_EIA-2012-15_AVX-P_Pad1.30x1.05mm_HandSolder
- removed the C4 at (243.5, 84.3)
- removed the C4 at (206.0, 37.0)
- removed R10: 3kR, up5k-synth:R_0805_2012Metric_Pad1.20x1.40mm_HandSolder
- removed R12: 1.8kR, up5k-synth:R_0805_2012Metric_Pad1.20x1.40mm_HandSolder
- removed R13: 10kR, up5k-synth:R_0805_2012Metric_Pad1.20x1.40mm_HandSolder
- removed R20, R22, R23, R25, R52, R57, R7: 360kR, up5k-synth:R_0805_2012Metric_Pad1.20x1.40mm_HandSolder
- removed R51: R_20mR_0603, up5k-synth:R_0603_1608Metric_Pad0.98x0.95mm_HandSolder
- removed R53, R54: R_16R_0603, up5k-synth:R_0603_1608Metric_Pad0.98x0.95mm_HandSolder
- removed R56: R_50kR_0603, up5k-synth:R_0603_1608Metric_Pad0.98x0.95mm_HandSolder
- added C2: 10uF_10V_0805, up5k-synth:C_0805_2012Metric_Pad1.18x1.45mm_HandSolder, F.Cu at (26.4, 225.7)
- added C25: 0.1uF_10V_0603, up5k-synth:C_0603_1608Metric_Pad1.08x0.95mm_HandSolder, F.Cu at (53.0, 221.0)
- added C26: 0.1uF_10V_0603, up5k-synth:C_0603_1608Metric_Pad1.08x0.95mm_HandSolder, F.Cu at (53.0, 218.5)
- added C29: 0.1uF_10V_0603, up5k-synth:C_0603_1608Metric_Pad1.08x0.95mm_HandSolder, F.Cu at (-91.0, 139.2)
- added C4: 10uF_10V_0805, up5k-synth:C_0805_2012Metric_Pad1.18x1.45mm_HandSolder, F.Cu at (31.9, 222.8)
- added U18: STP16CPC26PTR, up5k-synth:QSOP-24_3.9x8.7mm_P0.635mm, B.Cu at (198.9, 74.5)
- added U19: STP16CPC26PTR, up5k-synth:QSOP-24_3.9x8.7mm_P0.635mm, B.Cu at (186.0, 74.0)
- C1, C10, C11, C12, C13, C14, C15, C23, C24, C3, C31, C41, C42, C43, C44, C5, C6, C7, C8, C9, L1, L2, R1, R11, R16, R17, R18, R19, R2, R21, R24, R26, R27, R28, R29, R3, R30, R31, R32, R33, R34, R35, R36, R37, R38, R39, R4, R40, R41, R42, R43, R44, R45, R46, R47, R48, R49, R50, R58, R63, R84, R9, R93, R94: moved to F.Cu
- C16: value 27pF_10V_0603 -> 0.1uF_10V_0603; moved to F.Cu
- C17, C20, C21: value 4.7uF_10V_0805 -> 0.1uF_10V_0603; footprint up5k-synth:C_0805_2012Metric_Pad1.18x1.45mm_HandSolder -> up5k-synth:C_0603_1608Metric_Pad1.08x0.95mm_HandSolder; moved to F.Cu
- C18: value 1.0uF_10V_0805 -> 0.1uF_10V_0603; footprint up5k-synth:C_0805_2012Metric_Pad1.18x1.45mm_HandSolder -> up5k-synth:C_0603_1608Metric_Pad1.08x0.95mm_HandSolder; moved to F.Cu
- C34, C36: value CP_270uF_10v_PXF -> 0.1uF_10V_0603; footprint up5k-synth:CP_Elec_6.3x5.8 -> up5k-synth:C_0603_1608Metric_Pad1.08x0.95mm_HandSolder; moved to F.Cu
- C47, C48, C49, C50: value 0.1uF_10V_0603 -> C_150pF_10V_0603
- C51, C52, C54, C55: value 0.1uF_10V_0603 -> CP_270uF_10v_PXF; footprint up5k-synth:C_0603_1608Metric_Pad1.08x0.95mm_HandSolder -> up5k-synth:CP_Elec_6.3x5.8
- C57: value 0.1uF_10V_0603 -> 1.0uF_10V_0805; footprint up5k-synth:C_0603_1608Metric_Pad1.08x0.95mm_HandSolder -> up5k-synth:C_0805_2012Metric_Pad1.18x1.45mm_HandSolder; moved to F.Cu
- C58, C59: value 0.1uF_10V_0603 -> 4.7uF_10V_0805; footprint up5k-synth:C_0603_1608Metric_Pad1.08x0.95mm_HandSolder -> up5k-synth:C_0805_2012Metric_Pad1.18x1.45mm_HandSolder; moved to F.Cu
- C60: value 0.1uF_10V_0603 -> 27pF_10V_0603; moved to F.Cu
- C61, C62: value C_150pF_10V_0603 -> 4.7uF_10V_0805; footprint up5k-synth:C_0603_1608Metric_Pad1.08x0.95mm_HandSolder -> up5k-synth:C_0805_2012Metric_Pad1.18x1.45mm_HandSolder; moved to F.Cu
- C63: value C_150pF_10V_0603 -> 10uF_10V_0805; footprint up5k-synth:C_0603_1608Metric_Pad1.08x0.95mm_HandSolder -> up5k-synth:C_0805_2012Metric_Pad1.18x1.45mm_HandSolder; moved to F.Cu
- C64: value C_150pF_10V_0603 -> 0.1uF_10V_0603; moved to F.Cu
- D1, D2: value LED -> WS2812B; footprint up5k-synth:LED_Cree-PLCC4_3.2x2.8mm_CCW -> up5k-synth:LED_WS2812B_PLCC4_5.0x5.0mm_P3.2mm
- D19, D20: value WS2812B -> LED; footprint up5k-synth:LED_WS2812B_PLCC4_5.0x5.0mm_P3.2mm -> up5k-synth:LED_Cree-PLCC4_3.2x2.8mm_CCW
- R5, R6: value 1kR -> R_4k3R_0603; footprint up5k-synth:R_0805_2012Metric_Pad1.20x1.40mm_HandSolder -> up5k-synth:R_0603_1608Metric_Pad0.98x0.95mm_HandSolder
- R55, R61, R62: value R_50kR_0603 -> 360kR; footprint up5k-synth:R_0603_1608Metric_Pad0.98x0.95mm_HandSolder -> up5k-synth:R_0805_2012Metric_Pad1.20x1.40mm_HandSolder; moved to F.Cu
- R59, R60: value R_16R_0603 -> 360kR; footprint up5k-synth:R_0603_1608Metric_Pad0.98x0.95mm_HandSolder -> up5k-synth:R_0805_2012Metric_Pad1.20x1.40mm_HandSolder; moved to F.Cu
- R68, R69, R70, R71: value 360kR -> R_36kR_0603; footprint up5k-synth:R_0805_2012Metric_Pad1.20x1.40mm_HandSolder -> up5k-synth:R_0603_1608Metric_Pad0.98x0.95mm_HandSolder
- R76, R77, R80, R81: value 360kR -> R_16R_0603; footprint up5k-synth:R_0805_2012Metric_Pad1.20x1.40mm_HandSolder -> up5k-synth:R_0603_1608Metric_Pad0.98x0.95mm_HandSolder
- R78, R79, R82, R83: value 360kR -> R_50kR_0603; footprint up5k-synth:R_0805_2012Metric_Pad1.20x1.40mm_HandSolder -> up5k-synth:R_0603_1608Metric_Pad0.98x0.95mm_HandSolder
- R8: value 180kR -> 360kR; moved to F.Cu
- R85, R86: value 360kR -> 1kR; moved to F.Cu
- R87: value 360kR -> 3kR; moved to F.Cu
- R88: value 360kR -> 1.8kR; moved to F.Cu
- R89: value R_36kR_0603 -> 10kR; footprint up5k-synth:R_0603_1608Metric_Pad0.98x0.95mm_HandSolder -> up5k-synth:R_0805_2012Metric_Pad1.20x1.40mm_HandSolder; moved to F.Cu
- R90: value R_36kR_0603 -> 360kR; footprint up5k-synth:R_0603_1608Metric_Pad0.98x0.95mm_HandSolder -> up5k-synth:R_0805_2012Metric_Pad1.20x1.40mm_HandSolder; moved to F.Cu
- R91: value R_36kR_0603 -> 180kR; footprint up5k-synth:R_0603_1608Metric_Pad0.98x0.95mm_HandSolder -> up5k-synth:R_0805_2012Metric_Pad1.20x1.40mm_HandSolder; moved to F.Cu
- R92: value R_36kR_0603 -> R_20mR_0603; moved to F.Cu
- SW10, SW11, SW12, SW13, SW14, SW15, SW16, SW17, SW18, SW19, SW20, SW21, SW22, SW23, SW24, SW25: value SW_Push -> PB86-A2; footprint up5k-synth:SW_Push_1P1T_NO_6x6mm_H9.5mm -> up5k-synth:PB86-A2
- U14: value 74HC165 -> LMS33460; footprint up5k-synth:SO-16_3.9x9.9mm_P1.27mm -> up5k-synth:SC-70-5
- U15: value 74HC165 -> BQ24074; footprint up5k-synth:SO-16_3.9x9.9mm_P1.27mm -> up5k-synth:QFN-16-1EP_3x3mm_P0.5mm_EP1.9x1.9mm_ThermalVias
- U16: value 74HC165 -> TPS62120DCNR; footprint up5k-synth:SO-16_3.9x9.9mm_P1.27mm -> up5k-synth:SOT-23-8_Handsoldering
- U17: value 74HC165 -> TPS63031; footprint up5k-synth:SO-16_3.9x9.9mm_P1.27mm -> up5k-synth:VSON-10-1EP_3x3mm_P0.5mm_EP1.2x2mm_ThermalVias
- U3: value DS1881 -> 74HC165; footprint up5k-synth:TSSOP-16_4.4x5mm_P0.65mm -> up5k-synth:SO-16_3.9x9.9mm_P1.27mm
- U4: value LMS33460 -> 74HC165; footprint up5k-synth:SC-70-5 -> up5k-synth:SO-16_3.9x9.9mm_P1.27mm
- U5: value TPS62120DCNR -> 74HC165; footprint up5k-synth:SOT-23-8_Handsoldering -> up5k-synth:SO-16_3.9x9.9mm_P1.27mm
- U6: value BQ24074 -> 74HC165; footprint up5k-synth:QFN-16-1EP_3x3mm_P0.5mm_EP1.9x1.9mm_ThermalVias -> up5k-synth:SO-16_3.9x9.9mm_P1.27mm
- U8: value TPS63031 -> DS1881; footprint up5k-synth:VSON-10-1EP_3x3mm_P0.5mm_EP1.2x2mm_ThermalVias -> up5k-synth:TSSOP-16_4.4x5mm_P0.65mm
- moved SW7 436.6 mm to (-190.0, 155.5), turned to 0 degrees
- moved SW8 431.9 mm to (-174.5, 156.0), turned to 0 degrees
- moved SW9 428.4 mm to (-160.5, 156.0), turned to 0 degrees
- moved C63 425.2 mm to (-198.4, 183.1)
- moved C62 419.2 mm to (-198.4, 186.1), turned to 0 degrees
- moved C61 417.2 mm to (-193.6, 183.8)
- moved R94 415.2 mm to (-158.2, 204.3), turned to 0 degrees
- moved R92 408.2 mm to (-177.4, 208.2), turned to 0 degrees
- moved C64 404.5 mm to (-173.0, 207.1), turned to 0 degrees
- moved R89 400.9 mm to (-172.4, 204.3), turned to 0 degrees
- moved R90 394.9 mm to (-167.7, 204.3), turned to 0 degrees
- moved R91 394.7 mm to (-162.9, 204.3), turned to 0 degrees
- moved R93 383.6 mm to (-134.4, 204.3)
- moved SW2 383.4 mm to (-190.0, 145.5), turned to 0 degrees
- moved SW3 377.8 mm to (-174.0, 144.5), turned to 0 degrees
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Connections:
- net /BUF0_L renamed /Analog Output/BUF0_L
- net /BUF0_R renamed /Analog Output/BUF0_R
- net /LED_DOUT renamed Net-(D12-Pad2)
- net Net-(D10-Pad2) renamed /LED_OUT
- C16 pad 1: +1V2 -> /IO/SW_BTN20
- C16 pad 2: Net-(C16-Pad2) -> GND
- C18 pad 1: VBUS -> +3V3
- C20 pad 1: +BATT -> /IO/SW_BTN16
- C21 pad 1: /Vout -> /IO/SW_BTN21
- C23 pad 1: Net-(C23-Pad1) -> /IO/SW_BTN17
- C31 pad 1: +3V3 -> /IO/SW_BTN18
- C34 pad 1: Net-(C34-Pad1) -> /IO/SW_BTN23
- C34 pad 2: /OUT1_L -> GND
- C36 pad 1: Net-(C36-Pad1) -> /IO/SW_BTN19
- C36 pad 2: /OUT1_R -> GND
- C43 pad 1: /SW_BTN1 -> GND
- C43 pad 2: GND -> +3V3
- C44 pad 1: /SW_BTN5 -> GND
- C44 pad 2: GND -> +3V3
- C47 pad 1: /SW_BTN17 -> /Analog Output/F_PDM0_R
- C48 pad 1: /SW_BTN21 -> /Analog Output/F_PDM1_R
- C49 pad 1: /SW_BTN2 -> /Analog Output/F_PDM0_L
- C50 pad 1: /SW_BTN6 -> /Analog Output/F_PDM1_L
- C51 pad 1: /SW_BTN10 -> Net-(C51-Pad1)
- C51 pad 2: GND -> /OUT0_L
- C52 pad 1: /SW_BTN14 -> Net-(C52-Pad1)
- C52 pad 2: GND -> /OUT0_R
- C53 pad 1: /SW_BTN18 -> +3V3
- C54 pad 1: /SW_BTN22 -> Net-(C54-Pad1)
- C54 pad 2: GND -> /OUT1_L
- C55 pad 1: /SW_BTN3 -> Net-(C55-Pad1)
- C55 pad 2: GND -> /OUT1_R
- C56 pad 1: /SW_BTN7 -> +3V3
- C57 pad 1: /SW_BTN11 -> VBUS
- C58 pad 1: /SW_BTN15 -> GND
- C58 pad 2: GND -> /Power Supply/Vout
- C59 pad 1: /SW_BTN19 -> +BATT
- C60 pad 1: /SW_BTN23 -> +1V2
- C60 pad 2: GND -> Net-(C60-Pad2)
- C61 pad 1: /F_PDM0_R -> +3V3
- C62 pad 1: /F_PDM0_L -> /Power Supply/Vout
- C63 pad 1: /F_PDM1_R -> +3V3
- C64 pad 1: /F_PDM1_L -> Net-(C64-Pad1)
- D1 pad 1: Net-(D1-Pad1) -> +3V3
- D1 pad 3: Net-(D1-Pad3) -> GND
- D1 pad 4: /!CHG -> /LED_DATA
- D19 pad 1: +3V3 -> Net-(D19-Pad1)
- D19 pad 3: GND -> Net-(D19-Pad3)
- D19 pad 4: Net-(D18-Pad2) -> /Power Supply/!CHG
- D2 pad 1: Net-(D2-Pad1) -> +3V3
- D2 pad 3: Net-(D2-Pad3) -> GND
- D2 pad 4: /!PGOOD -> Net-(D1-Pad2)
- D20 pad 1: +3V3 -> Net-(D20-Pad1)
- D20 pad 3: GND -> Net-(D20-Pad3)
- D20 pad 4: Net-(D19-Pad2) -> /Power Supply/!PGOOD
- D5 pad 4: /LED_DATA -> Net-(D2-Pad2)
- ENC1 pad 2: /SW_ENC1 -> /IO/SW_ENC1
- ENC1 pad 3: /ENC1_A -> /IO/ENC1_A
- ENC1 pad 5: /ENC1_B -> /IO/ENC1_B
- ENC2 pad 2: /SW_ENC2 -> /IO/SW_ENC2
- ENC2 pad 3: /ENC2_A -> /IO/ENC2_A
- ENC2 pad 5: /ENC2_B -> /IO/ENC2_B
- R11 pad 1: Net-(R11-Pad1) -> /IO/SW_BTN17
- R11 pad 2: +1V2 -> GND
- R19 pad 1: Net-(R19-Pad1) -> /IO/SW_BTN22
- R21 pad 1: Net-(R21-Pad1) -> /IO/SW_BTN18
- R24 pad 1: Net-(R24-Pad1) -> /IO/SW_BTN23
- R26 pad 1: Net-(R26-Pad1) -> /IO/SW_BTN19
- R3 pad 1: /BGD -> /IO/SW_BTN20
- R3 pad 2: /PSU_EN -> GND
- R5 pad 1: /Vout -> GND
- R5 pad 2: Net-(D1-Pad2) -> Net-(R5-Pad2)
- R55 pad 1: /OUT0_L -> Net-(R55-Pad1)
- R55 pad 2: GND -> +3V3
- R58 pad 1: /SW_BTN8 -> Net-(R58-Pad1)
- R59 pad 2: Net-(C34-Pad1) -> GND
- R6 pad 1: /Vout -> GND
- R6 pad 2: Net-(D2-Pad2) -> Net-(R6-Pad2)
- R60 pad 2: Net-(C36-Pad1) -> GND
- R61 pad 1: /OUT1_L -> Net-(R61-Pad1)
- R62 pad 1: /OUT1_R -> /IO/SW_ENC1
- R63 pad 1: /SW_BTN12 -> /IO/SW_ENC1
- R64 pad 1: /SW_BTN16 -> Net-(R64-Pad1)
- R65 pad 1: /SW_BTN20 -> Net-(R65-Pad1)
- R66 pad 1: /SW_BTN1 -> Net-(R66-Pad1)
- R67 pad 1: /SW_BTN5 -> Net-(R67-Pad1)
- R68 pad 1: /SW_BTN9 -> /PDM0_R
- R68 pad 2: GND -> /Analog Output/F_PDM0_R
- R69 pad 1: /SW_BTN13 -> /PDM1_R
- R69 pad 2: GND -> /Analog Output/F_PDM1_R
- R70 pad 1: /SW_BTN17 -> /PDM0_L
- R70 pad 2: GND -> /Analog Output/F_PDM0_L
- R71 pad 1: /SW_BTN21 -> /PDM1_L
- R71 pad 2: GND -> /Analog Output/F_PDM1_L
- R73 pad 1: /SW_BTN2 -> Net-(R73-Pad1)
- R74 pad 1: /SW_BTN6 -> Net-(R74-Pad1)
- R75 pad 1: /SW_BTN10 -> Net-(R75-Pad1)
- R76 pad 1: /SW_BTN14 -> Net-(R76-Pad1)
- R76 pad 2: GND -> Net-(C51-Pad1)
- R77 pad 1: /SW_BTN18 -> Net-(R77-Pad1)
- R77 pad 2: GND -> Net-(C52-Pad1)
- R78 pad 1: /SW_BTN22 -> /OUT0_L
- R79 pad 1: /SW_BTN3 -> /OUT0_R
- R8 pad 1: +1V2 -> /IO/SW_BTN16
- R8 pad 2: Net-(C16-Pad2) -> GND
- R80 pad 1: /SW_BTN7 -> Net-(R80-Pad1)
- R80 pad 2: GND -> Net-(C54-Pad1)
- R81 pad 1: /SW_BTN11 -> Net-(R81-Pad1)
- R81 pad 2: GND -> Net-(C55-Pad1)
- R82 pad 1: /SW_BTN15 -> /OUT1_L
- R83 pad 1: /SW_BTN19 -> /OUT1_R
- R84 pad 1: /SW_BTN23 -> /Power Supply/BGD
- R84 pad 2: GND -> /PSU_EN
- R85 pad 1: Net-(R85-Pad1) -> /Power Supply/Vout
- R85 pad 2: GND -> Net-(D19-Pad2)
- R86 pad 1: Net-(R86-Pad1) -> /Power Supply/Vout
- R86 pad 2: GND -> Net-(D20-Pad2)
- R87 pad 1: Net-(R87-Pad1) -> GND
- R87 pad 2: GND -> Net-(R87-Pad2)
- R88 pad 1: Net-(R88-Pad1) -> GND
- R88 pad 2: GND -> Net-(R88-Pad2)
- R89 pad 1: /PDM0_R -> Net-(R89-Pad1)
- R89 pad 2: /F_PDM0_R -> GND
- R9 pad 1: GND -> /IO/SW_BTN21
- R9 pad 2: Net-(C16-Pad2) -> GND
- R90 pad 1: /PDM0_L -> Net-(R90-Pad1)
- R90 pad 2: /F_PDM0_L -> +3V3
- R91 pad 1: /PDM1_R -> +1V2
- R91 pad 2: /F_PDM1_R -> Net-(C60-Pad2)
- R92 pad 1: /PDM1_L -> -BATT
- R92 pad 2: /F_PDM1_L -> GND
- R93 pad 1: /SW_ENC1 -> GND
- R93 pad 2: GND -> Net-(C60-Pad2)
- R94 pad 1: /SW_ENC1 -> Net-(R94-Pad1)
- R94 pad 2: GND -> +1V2
- SW10 pad 1: +3V3 -> /IO/SW_BTN0
- SW10 pad 2: /SW_BTN18 -> +3V3
- SW11 pad 1: +3V3 -> /IO/SW_BTN1
- SW11 pad 2: /SW_BTN3 -> +3V3
- SW12 pad 1: +3V3 -> /IO/SW_BTN2
- SW12 pad 2: /SW_BTN11 -> +3V3
- SW13 pad 1: +3V3 -> /IO/SW_BTN3
- SW13 pad 2: /SW_BTN19 -> +3V3
- SW14 pad 1: +3V3 -> /IO/SW_BTN4
- SW14 pad 2: /SW_BTN4 -> +3V3
- SW15 pad 1: +3V3 -> /IO/SW_BTN5
- SW15 pad 2: /SW_BTN12 -> +3V3
- SW16 pad 1: +3V3 -> /IO/SW_BTN6
- SW16 pad 2: /SW_BTN20 -> +3V3
- SW17 pad 1: +3V3 -> /IO/SW_BTN7
- SW17 pad 2: /SW_BTN5 -> +3V3
- SW18 pad 1: +3V3 -> /IO/SW_BTN8
- SW18 pad 2: /SW_BTN13 -> +3V3
- SW19 pad 1: +3V3 -> /IO/SW_BTN9
- SW19 pad 2: /SW_BTN21 -> +3V3
- SW2 pad 2: /SW_BTN0 -> /IO/SW_BTN16
- SW20 pad 1: +3V3 -> /IO/SW_BTN10
- SW20 pad 2: /SW_BTN6 -> +3V3
- SW21 pad 1: +3V3 -> /IO/SW_BTN11
- SW21 pad 2: /SW_BTN14 -> +3V3
- SW22 pad 1: +3V3 -> /IO/SW_BTN12
- SW22 pad 2: /SW_BTN22 -> +3V3
- SW23 pad 1: +3V3 -> /IO/SW_BTN13
- SW23 pad 2: /SW_BTN7 -> +3V3
- SW24 pad 1: +3V3 -> /IO/SW_BTN14
- SW24 pad 2: /SW_BTN15 -> +3V3
- SW25 pad 1: +3V3 -> /IO/SW_BTN15
- SW25 pad 2: /SW_BTN23 -> +3V3
- SW3 pad 2: /SW_BTN8 -> /IO/SW_BTN17
- SW4 pad 2: /SW_BTN16 -> /IO/SW_BTN18
- SW5 pad 2: /SW_BTN1 -> /IO/SW_BTN19
- SW6 pad 2: /SW_BTN9 -> /IO/SW_BTN20
- SW7 pad 2: /SW_BTN17 -> /IO/SW_BTN21
- SW8 pad 2: /SW_BTN2 -> /IO/SW_BTN22
- SW9 pad 2: /SW_BTN10 -> /IO/SW_BTN23
- U10 pad 1: Net-(R53-Pad1) -> Net-(R76-Pad1)
- U10 pad 2: Net-(R53-Pad1) -> Net-(R76-Pad1)
- U10 pad 6: Net-(R54-Pad1) -> Net-(R77-Pad1)
- U10 pad 7: Net-(R54-Pad1) -> Net-(R77-Pad1)
- U11 pad 1: Net-(R59-Pad1) -> Net-(R80-Pad1)
- U11 pad 2: Net-(R59-Pad1) -> Net-(R80-Pad1)
- U11 pad 3: /BUF1_L -> /Analog Output/BUF1_L
- U11 pad 5: /BUF1_R -> /Analog Output/BUF1_R
- U11 pad 6: Net-(R60-Pad1) -> Net-(R81-Pad1)
- U11 pad 7: Net-(R60-Pad1) -> Net-(R81-Pad1)
- U14 pad 1: /SW_LOAD -> Net-(U14-Pad1)
- U14 pad 2: /SW_CLK -> GND
- U14 pad 3: /SW_BTN4 -> GND
- U14 pad 4: /SW_BTN5 -> /Power Supply/BGD
- U14 pad 5: /SW_BTN6 -> /PSU_EN
- U15 pad 1: /SW_LOAD -> Net-(R89-Pad1)
- U15 pad 10: Net-(U14-Pad9) -> /Power Supply/Vout
- U15 pad 11: /SW_BTN8 -> /Power Supply/Vout
- U15 pad 12: /SW_BTN9 -> Net-(R87-Pad2)
- U15 pad 13: /SW_BTN10 -> VBUS
- U15 pad 14: /SW_BTN11 -> GND
- U15 pad 15: Net-(R86-Pad1) -> Net-(U15-Pad15)
- U15 pad 16: +3V3 -> Net-(R88-Pad2)
- U15 pad 2: /SW_CLK -> +BATT
- U15 pad 3: /SW_BTN12 -> +BATT
- U15 pad 4: /SW_BTN13 -> GND
- U15 pad 5: /SW_BTN14 -> GND
- U15 pad 6: /SW_BTN15 -> /Power Supply/Vout
- U15 pad 7: Net-(U15-Pad7) -> /Power Supply/!PGOOD
- U15 pad 9: Net-(U15-Pad9) -> /Power Supply/!CHG
- U16 pad 1: /SW_LOAD -> +3V3
- U16 pad 2: /SW_CLK -> GND
- U16 pad 3: /SW_BTN20 -> Net-(R90-Pad1)
- U16 pad 4: /SW_BTN21 -> +1V2
- U16 pad 5: /SW_BTN22 -> Net-(C60-Pad2)
- U16 pad 6: /SW_BTN23 -> Net-(R94-Pad1)
- U16 pad 7: Net-(U16-Pad7) -> Net-(L1-Pad1)
- U16 pad 8: GND -> +1V2
- U17 pad 1: /SW_LOAD -> +3V3
- U17 pad 10: Net-(U16-Pad9) -> +3V3
- U17 pad 11: /SW_ENC1 -> (no net)
- U17 pad 2: /SW_CLK -> Net-(L2-Pad2)
- U17 pad 3: /SW_ENC2 -> GND
- U17 pad 4: /ENC2_A -> Net-(L2-Pad1)
- U17 pad 5: /ENC2_B -> /Power Supply/Vout
- U17 pad 6: Net-(U17-Pad6) -> /Power Supply/BGD
- U17 pad 7: Net-(U17-Pad7) -> Net-(C64-Pad1)
- U17 pad 8: GND -> Net-(C64-Pad1)
- U17 pad 9: /SW_DATA -> GND
- U3 pad 1: GND -> /SW_LOAD
- U3 pad 10: /F_PDM1_R -> Net-(R55-Pad1)
- U3 pad 11: /BUF1_R -> /IO/SW_BTN0
- U3 pad 12: Net-(R20-Pad1) -> /IO/SW_BTN1
- U3 pad 13: /SC0_SDA_PAD[0] -> /IO/SW_BTN2
- U3 pad 14: /SC0_SCL_PAD[1] -> /IO/SW_BTN3
- U3 pad 15: +3V3 -> Net-(R58-Pad1)
- U3 pad 16: GND -> +3V3
- U3 pad 2: Net-(R22-Pad1) -> /SW_CLK
- U3 pad 3: Net-(R21-Pad1) -> /IO/SW_BTN4
- U3 pad 4: Net-(U3-Pad4) -> /IO/SW_BTN5
- U3 pad 5: Net-(R19-Pad1) -> /IO/SW_BTN6
- U3 pad 6: /BUF1_L -> /IO/SW_BTN7
- U3 pad 7: GND -> Net-(U3-Pad7)
- U3 pad 8: /F_PDM1_L -> GND
- U3 pad 9: GND -> Net-(U3-Pad9)
- U4 pad 1: Net-(U4-Pad1) -> /SW_LOAD
- U4 pad 2: GND -> /SW_CLK
- U4 pad 3: GND -> /IO/SW_BTN12
- U4 pad 4: /BGD -> /IO/SW_BTN13
- U4 pad 5: /PSU_EN -> /IO/SW_BTN14
- U5 pad 1: +3V3 -> /SW_LOAD
- U5 pad 2: GND -> /SW_CLK
- U5 pad 3: Net-(R7-Pad1) -> /IO/SW_BTN20
- U5 pad 4: +1V2 -> /IO/SW_BTN21
- U5 pad 5: Net-(C16-Pad2) -> /IO/SW_BTN22
- U5 pad 6: Net-(R11-Pad1) -> /IO/SW_BTN23
- U5 pad 7: Net-(L1-Pad1) -> Net-(U5-Pad7)
- U5 pad 8: +1V2 -> GND
- U6 pad 1: Net-(R13-Pad1) -> /SW_LOAD
- U6 pad 10: /Vout -> Net-(U5-Pad9)
- U6 pad 11: /Vout -> /IO/SW_ENC1
- U6 pad 12: Net-(R10-Pad2) -> /IO/ENC1_A
- U6 pad 13: VBUS -> /IO/ENC1_B
- U6 pad 14: GND -> Net-(U6-Pad14)
- U6 pad 15: Net-(U6-Pad15) -> Net-(R61-Pad1)
- U6 pad 16: Net-(R12-Pad2) -> +3V3
- U6 pad 2: +BATT -> /SW_CLK
- U6 pad 3: +BATT -> /IO/SW_ENC2
- U6 pad 4: GND -> /IO/ENC2_A
- U6 pad 5: GND -> /IO/ENC2_B
- U6 pad 6: /Vout -> Net-(U6-Pad6)
- U6 pad 7: /!PGOOD -> Net-(U6-Pad7)
- U6 pad 9: /!CHG -> /SW_DATA
- U8 pad 1: +3V3 -> GND
- U8 pad 10: +3V3 -> /Analog Output/F_PDM1_R
- U8 pad 11: (no net) -> /Analog Output/BUF1_R
- U8 pad 2: Net-(L2-Pad2) -> Net-(R67-Pad1)
- U8 pad 3: GND -> Net-(R66-Pad1)
- U8 pad 4: Net-(L2-Pad1) -> Net-(U8-Pad4)
- U8 pad 5: /Vout -> Net-(R64-Pad1)
- U8 pad 6: /BGD -> /Analog Output/BUF1_L
- U8 pad 7: Net-(C23-Pad1) -> GND
- U8 pad 8: Net-(C23-Pad1) -> /Analog Output/F_PDM1_L
- U9 pad 10: /F_PDM0_R -> /Analog Output/F_PDM0_R
- U9 pad 12: Net-(R24-Pad1) -> Net-(R73-Pad1)
- U9 pad 2: Net-(R26-Pad1) -> Net-(R75-Pad1)
- U9 pad 3: Net-(R25-Pad1) -> Net-(R74-Pad1)
- U9 pad 5: Net-(R23-Pad1) -> Net-(R72-Pad1)
- U9 pad 8: /F_PDM0_L -> /Analog Output/F_PDM0_L

Commit message: Design checkpoint at 20210701
Parts:
- C1, C10, C11, C12, C13, C14, C15, C2, C24, C3, C4, C5, C57, C58, C59, C6, C60, C61, C62, C64, C7, C8, C9, L1, L2, R16, R17, R18, R4, R84, R85, R86, R87, R88, R89, R90, R91, R92, R93, R94: moved to B.Cu
- U13: moved to F.Cu
- moved C61 503.8 mm to (295.1, 61.2)
- moved R90 484.1 mm to (293.6, 57.2), turned to 90 degrees
- moved C60 474.8 mm to (282.1, 57.7), turned to 270 degrees
- moved R91 473.8 mm to (288.6, 60.7), turned to 180 degrees
- moved R94 466.4 mm to (284.1, 56.2), turned to 90 degrees
- moved SW3 444.0 mm to (269.0, 115.0), turned to 90 degrees
- moved R93 439.0 mm to (280.1, 59.7), turned to 90 degrees
- moved SW9 353.5 mm to (178.2, 55.0), turned to 90 degrees
- moved R92 335.0 mm to (113.5, 42.2), turned to 270 degrees
- moved C62 330.0 mm to (101.0, 47.2), turned to 180 degrees
- moved C64 319.0 mm to (97.0, 37.2), turned to 90 degrees
- moved C57 315.8 mm to (78.5, 28.8)
- moved SW6 315.3 mm to (178.2, 72.5), turned to 270 degrees
- moved R88 315.0 mm to (84.0, 28.2)
- moved C58 312.3 mm to (80.5, 38.2)
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Connections:
- U1 pad 88: (no net) -> Net-(C7-Pad1)
Routing:
- net /MII_GRXCK: track 0.00 -> 52.0 mm, vias 0 -> 2
- net /SDHC1_DAT[0]: track 0.00 -> 42.7 mm
- net /SDHC1_SDCLK: track 0.00 -> 38.6 mm
- net /SDHC1_SDCMD: track 0.00 -> 34.5 mm
- net /MII_GCOL: track 0.00 -> 33.9 mm, vias 0 -> 2
- net /SDHC1_DAT[3]: track 0.00 -> 33.7 mm
- net /SDHC1_DAT[1]: track 0.00 -> 32.7 mm
- net /SDHC1_DAT[2]: track 0.00 -> 29.2 mm
- net GND: track 0.00 -> 27.6 mm, vias 0 -> 3
- net /D-: track 0.00 -> 24.9 mm
- net /D+: track 0.00 -> 24.8 mm
- net /MII_GTX[3]: track 0.00 -> 21.3 mm
- net /MII_GRDV: track 0.00 -> 20.9 mm, vias 0 -> 2
- net /MII_GTXER: track 0.00 -> 19.9 mm, vias 0 -> 2
- net /MII_GTX[2]: track 0.00 -> 19.8 mm
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Other:
- net class MII interface added: clearance 0.127, trace_width 0.127, via_dia 0.8, via_drill 0.4
- net class USB Data added: clearance 0.1524, trace_width 0.2, via_dia 0.8, via_drill 0.4
- net class config spi bus added: clearance 0.127, trace_width 0.127, via_dia 0.8, via_drill 0.4
- rule trace_min: 0.2 -> 0.127

Commit message: Design checkpoint at 20210702
Parts:
- moved U12 33.8 mm to (89.8, 15.2)
- moved R88 20.5 mm to (72.7, 45.4), turned to 180 degrees
- moved R89 20.2 mm to (69.1, 42.0)
- moved C59 16.5 mm to (69.2, 37.4), turned to 90 degrees
- moved C57 15.7 mm to (78.2, 44.5), turned to 270 degrees
- moved R87 10.2 mm to (81.0, 41.7), turned to 180 degrees
- moved L2 10.0 mm to (100.0, 43.2), turned to 0 degrees
- moved C62 9.62 mm to (96.5, 38.8), turned to 90 degrees
- moved U15 8.79 mm to (75.2, 39.9), turned to 0 degrees
- moved U14 8.16 mm to (93.8, 34.5), turned to 270 degrees
- moved R84 7.94 mm to (89.3, 34.4), turned to 90 degrees
- moved SW3 7.29 mm to (265.2, 108.8)
- moved D1 6.25 mm to (103.5, 61.2)
- moved D2 6.16 mm to (95.7, 61.2)
- moved D5 6.15 mm to (87.8, 61.2)
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Routing:
- net VBUS: track 0.00 -> 99.3 mm, vias 0 -> 1
- net GND: track 27.6 -> 70.6 mm, vias 3 -> 4
- net +BATT: track 0.00 -> 32.7 mm
- net /Power Supply/Vout: track 0.00 -> 25.8 mm
- net Net-(R88-Pad2): track 0.00 -> 5.25 mm
- net Net-(R89-Pad1): track 0.00 -> 4.82 mm
- net /Power Supply/BGD: track 0.00 -> 3.78 mm
- net Net-(R87-Pad2): track 0.00 -> 3.72 mm
- net /PSU_EN: track 0.00 -> 3.70 mm
- net Net-(L2-Pad2): track 0.00 -> 2.58 mm
- net Net-(L2-Pad1): track 0.00 -> 2.22 mm
- net /D-: track 24.9 -> 24.3 mm
- added copper zone on F.Cu, net GND
Other:
- net class Default: clearance 0.2 -> 0.127
- rule trace_clearance: 0.2 -> 0.127

Commit message: Design checkpoint on 20210706
Parts:
- moved C61 186.0 mm to (113.5, 20.8), turned to 270 degrees
- moved R91 180.6 mm to (114.0, 14.3), turned to 90 degrees
- moved R90 180.1 mm to (117.5, 19.3), turned to 0 degrees
- moved U16 176.8 mm to (117.0, 14.1), turned to 90 degrees
- moved R93 173.6 mm to (115.0, 5.80), turned to 0 degrees
- moved C60 172.4 mm to (117.0, 7.80), turned to 180 degrees
- moved R94 171.9 mm to (118.5, 9.80), turned to 0 degrees
- moved L1 170.7 mm to (122.5, 14.8), turned to 270 degrees
- moved U7 155.4 mm to (135.0, 58.0), turned to 90 degrees
- moved D4 0.52 mm to (176.2, 35.0)
- moved C64 0.50 mm to (100.8, 34.8), turned to 0 degrees
Routing:
- net GND: track 70.6 -> 110.5 mm, vias 4 -> 12
- net /Power Supply/BGD: track 3.78 -> 11.5 mm
- net Net-(C64-Pad1): track 0.00 -> 5.57 mm
- net VBUS: track 99.3 -> 104.3 mm, vias 1 -> 2
- net +3V3: track 11.2 -> 15.6 mm
- net /D-: track 24.3 -> 25.5 mm
- net /D+: track 25.1 -> 26.1 mm
- added copper zone on B.Cu, net GND
Other:
- board outline added: 250 x 100 mm

Commit message: Design checkpoint of 20210707
Parts:
- moved U19 88.3 mm to (216.5, 86.2), turned to 90 degrees
- moved U18 83.8 mm to (239.5, 85.8), turned to 90 degrees
- moved C34 64.6 mm to (10.5, 180.5)
- moved C43 63.8 mm to (18.0, 176.8)
- moved C42 60.5 mm to (10.8, 176.2)
- moved C63 53.4 mm to (13.2, 172.0)
- moved C41 50.2 mm to (22.7, 168.0)
- moved C20 50.2 mm to (20.5, 170.5)
- moved C44 39.7 mm to (3.00, 169.2)
- moved C17 34.5 mm to (15.8, 161.8)
- moved U12 33.3 mm to (109.5, 42.0), turned to 270 degrees
- moved C26 32.4 mm to (16.8, 155.2)
- moved C21 31.6 mm to (24.8, 152.8)
- moved C16 31.1 mm to (18.8, 142.0)
- moved C25 30.9 mm to (20.5, 147.0)
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Connections:
- P2 pad 2: /ADC0IN[12] -> /ADC1IN[5]
- P21 pad 2: /ADC1IN[10] -> /ADC0IN[15]
- P22 pad 2: /ADC1IN[4] -> /ADC0IN[14]
- P23 pad 2: /ADC1IN[11] -> /ADC0IN[13]
- P24 pad 2: /ADC1IN[5] -> /ADC0IN[12]
- P4 pad 2: /ADC0IN[13] -> /ADC1IN[11]
- P6 pad 2: /ADC0IN[14] -> /ADC1IN[4]
- P8 pad 2: /ADC0IN[15] -> /ADC1IN[10]
Routing:
- net /CDONE: track 3.16 -> 70.5 mm, vias 1 -> 2
- net +BATT: track 32.7 -> 99.4 mm
- net +1V2: track 4.41 -> 31.7 mm, vias 1 -> 4
- net +3V3: track 15.6 -> 39.5 mm, vias 0 -> 3
- net GND: track 110.5 -> 128.1 mm, vias 12 -> 14
- net /MII_GMDIO: track 6.54 -> 22.9 mm
- net /CLK48M: track 0.00 -> 10.5 mm
- net Net-(D13-Pad2): track 0.00 -> 9.76 mm, vias 0 -> 1
- net -BATT: track 0.00 -> 7.99 mm
- net /MII_GRXCK: track 52.0 -> 46.5 mm
- net /PDM0_R: track 0.00 -> 5.20 mm
- net /PDM0_L: track 0.00 -> 3.49 mm
- net /PMOD[6]: track 0.00 -> 1.66 mm, vias 0 -> 1

Commit message: Design checkpoint at 20210712
Parts:
- R5, R55, R59, R6: moved to B.Cu
- moved R8 268.8 mm to (242.8, 29.5)
- moved R55 267.5 mm to (240.8, 34.0), turned to 90 degrees
- moved R6 263.6 mm to (242.8, 86.1), turned to 180 degrees
- moved R58 260.3 mm to (244.0, 35.8), turned to 90 degrees
- moved R5 252.0 mm to (220.0, 87.0), turned to 90 degrees
- moved R59 239.6 mm to (233.2, 91.2), turned to 90 degrees
- moved SW1 192.0 mm to (41.5, 33.5)
- moved U3 142.1 mm to (234.6, 37.8)
- moved U5 142.0 mm to (42.0, 73.8)
- moved U6 112.9 mm to (92.0, 68.2)
- moved U4 94.0 mm to (224.2, 85.8)
- moved U18 24.6 mm to (215.0, 83.2), turned to 0 degrees
- moved U19 19.5 mm to (235.8, 83.2), turned to 0 degrees
- moved R2 17.0 mm to (170.2, 62.5)
- moved DIS1 14.3 mm to (142.8, 81.8)
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Connections:
- net Net-(U1-Pad32) renamed /DISPLAY_CMD
- DIS1 pad 3: Net-(DIS1-Pad3) -> /SC4_SCK_PAD[1]
- DIS1 pad 4: Net-(DIS1-Pad4) -> /SC4_PAD[0]
- U1 pad 33: Net-(U1-Pad33) -> /DISPLAY_CS
- U1 pad 78: Net-(U1-Pad78) -> /SEQ_OE
- U1 pad 79: Net-(U1-Pad79) -> /SEQ_LE
- U1 pad 85: Net-(U1-Pad85) -> /SEQ_DATA
- U1 pad 86: Net-(U1-Pad86) -> /SEQ_CLK
- U18 pad 2: /IO/SEQ_DATA -> /SEQ_DATA
- U18 pad 21: /IO/SEQ_OE -> /SEQ_OE
- U18 pad 3: /IO/SEQ_CLK -> /SEQ_CLK
- U18 pad 4: /IO/SEQ_LE -> /SEQ_LE
- U19 pad 21: /IO/SEQ_OE -> /SEQ_OE
- U19 pad 3: /IO/SEQ_CLK -> /SEQ_CLK
- U19 pad 4: /IO/SEQ_LE -> /SEQ_LE
Routing:
- net Net-(R6-Pad2): track 0.00 -> 3.49 mm

Commit message: Design checkpoint on 20210713
Parts:
- added C19: 0.1uF_10V_0603, up5k-synth:C_0603_1608Metric_Pad1.08x0.95mm_HandSolder, F.Cu at (121.0, 158.8)
- added C22: 0.1uF_10V_0603, up5k-synth:C_0603_1608Metric_Pad1.08x0.95mm_HandSolder, F.Cu at (125.8, 155.4)
- added C27: C_47uF_0805, up5k-synth:C_0805_2012Metric_Pad1.18x1.45mm_HandSolder, F.Cu at (116.4, 156.0)
- added C28: C_47uF_0805, up5k-synth:C_0805_2012Metric_Pad1.18x1.45mm_HandSolder, F.Cu at (122.4, 152.7)
- added C30: C_220uF_1206, up5k-synth:C_1206_3216Metric_Pad1.33x1.80mm_HandSolder, F.Cu at (111.0, 152.9)
- added C32: C_220uF_1206, up5k-synth:C_1206_3216Metric_Pad1.33x1.80mm_HandSolder, F.Cu at (111.0, 156.2)
- added C33: C_47uF_0805, up5k-synth:C_0805_2012Metric_Pad1.18x1.45mm_HandSolder, F.Cu at (138.4, 41.6)
- added C35: C_47uF_0805, up5k-synth:C_0805_2012Metric_Pad1.18x1.45mm_HandSolder, F.Cu at (146.4, 38.8)
- added C37: C_220uF_1206, up5k-synth:C_1206_3216Metric_Pad1.33x1.80mm_HandSolder, F.Cu at (134.6, 41.0)
- added C38: C_220uF_1206, up5k-synth:C_1206_3216Metric_Pad1.33x1.80mm_HandSolder, F.Cu at (149.6, 37.4)
- C17, C18, C42: moved to B.Cu
- R80, R81, R82, R83, U11: moved to F.Cu
- moved C18 283.2 mm to (268.3, 37.8)
- moved C42 228.7 mm to (223.8, 93.0)
- moved C17 210.7 mm to (214.2, 91.0)
- moved R67 168.2 mm to (161.8, 44.3), turned to 0 degrees
- moved R66 165.9 mm to (158.3, 46.3), turned to 180 degrees
- moved R64 162.5 mm to (156.8, 44.3), turned to 180 degrees
- moved R69 156.4 mm to (151.6, 49.5)
- moved C48 156.2 mm to (152.5, 47.0)
- moved C50 156.1 mm to (148.9, 47.0)
- moved R71 156.1 mm to (149.8, 49.5)
- moved U8 147.8 mm to (146.2, 41.8), turned to 180 degrees
- moved R65 136.9 mm to (138.4, 41.0), turned to 90 degrees
- moved U11 134.7 mm to (143.6, 44.6), turned to 270 degrees
- moved R80 96.2 mm to (136.8, 44.9), turned to 90 degrees
- moved R82 78.9 mm to (139.2, 38.4)
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Connections:
- R76 pad 2: Net-(C51-Pad1) -> Net-(C28-Pad2)
- R77 pad 2: Net-(C52-Pad1) -> Net-(C27-Pad2)
- R80 pad 2: Net-(C54-Pad1) -> Net-(C33-Pad2)
- R81 pad 2: Net-(C55-Pad1) -> Net-(C35-Pad2)
- U8 pad 10: /Analog Output/F_PDM1_R -> /Analog Output/F_PDM1_L
- U8 pad 11: /Analog Output/BUF1_R -> /Analog Output/BUF1_L
- U8 pad 6: /Analog Output/BUF1_L -> /Analog Output/BUF1_R
- U8 pad 8: /Analog Output/F_PDM1_L -> /Analog Output/F_PDM1_R
Routing:
- net VBUS: track 104.3 -> 113.7 mm
- net /PDM1_R: track 0.00 -> 5.96 mm
- net /PDM1_L: track 0.00 -> 5.42 mm
- net /PDM0_R: track 5.20 -> 0.00 mm
- net /PDM0_L: track 3.49 -> 0.00 mm
- net Net-(R6-Pad2): track 3.49 -> 0.00 mm
- net /Analog Output/F_PDM1_L: track 0.00 -> 1.67 mm
- net /Analog Output/F_PDM1_R: track 0.00 -> 1.60 mm
- net /CDONE: track 70.5 -> 72.0 mm
