File: gf-minus1/gf-minus1.kicad_pcb (KiCad board)
At the start: 4 copper layers, 100 x 100 mm, 109 parts, among them J1 MEM2061-01-188-00-A, J2 10118194-0001LF, J3 PMOD_conn, J4 debug_conn, J5 AudioJack3_SwitchTR, J6 AudioJack3_SwitchTR, SW1 SW_Push, SW26 SW_DPDT_x2_MFS201N−16−Z, U1 ATSAME53N19A, U10 AD8531, U11 AD8531, U12 DS2745, U13 DSC6003JI2A, U14 LMS33460, U15 BQ24074, U16 TPS62120DCNR, U17 TPS63031, U2 DRA818_iCE40-UP5K-SG48, U7 DSC6003JI2A, U8 DS1881, U9 DS1881

Commit message: GF-MINUS1 progress
Parts:
- moved C53 13.7 mm to (117.3, 58.2), turned to 0 degrees
- moved C56 7.40 mm to (129.5, 73.5), turned to 180 degrees
- moved D3 7.34 mm to (72.2, 59.2)
- moved C61 7.27 mm to (110.1, 111.3), turned to 90 degrees
- moved R93 6.20 mm to (106.7, 108.7)
- moved R87 5.20 mm to (79.9, 118.2), turned to 270 degrees
- moved C58 5.02 mm to (79.9, 122.4), turned to 90 degrees
- moved R92 4.47 mm to (102.2, 125.0)
- moved C57 4.20 mm to (75.4, 116.8)
- moved C1 3.95 mm to (85.8, 90.0), turned to 180 degrees
- moved D4 3.22 mm to (68.8, 59.2), turned to 180 degrees
- moved R78 3.17 mm to (140.9, 76.4), turned to 180 degrees
- moved R90 3.13 mm to (113.8, 115.3)
- moved R76 2.73 mm to (134.5, 81.6)
- moved C24 2.55 mm to (63.8, 92.0)
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Connections:
- C47 pad 1: /Analog Output/F_PDM0_R -> /Analog Output/F_PDM0_L
- C49 pad 1: /Analog Output/F_PDM0_L -> /Analog Output/F_PDM0_R
- R68 pad 1: /PDM0_R -> /PDM0_L
- R68 pad 2: /Analog Output/F_PDM0_R -> /Analog Output/F_PDM0_L
- R70 pad 1: /PDM0_L -> /PDM0_R
- R70 pad 2: /Analog Output/F_PDM0_L -> /Analog Output/F_PDM0_R
- U1 pad 48: /MII_GRXCK -> /MII_GTXCK
- U2 pad 18: /MII_GMDC -> /MII_GMDIO
- U2 pad 19: /MII_GMDIO -> /MII_GMDC
- U2 pad 2: /MII_GCRS -> /MII_GTX[2]
- U2 pad 3: /MII_GTEN -> /MII_GTX[3]
- U2 pad 37: /PDM0_L -> /PDM0_R
- U2 pad 38: /PDM0_R -> /PDM0_L
- U2 pad 45: /MII_GTX[3] -> /MII_GCRS
- U2 pad 46: /MII_GTX[2] -> /MII_GTEN
- U2 pad 47: /MII_GTX[1] -> /MII_GTX[0]
- U2 pad 48: /MII_GTX[0] -> /MII_GTX[1]
- U2 pad 9: /MII_GRXER -> /MII_GTXCK
- U9 pad 10: /Analog Output/F_PDM0_L -> /Analog Output/F_PDM0_R
- U9 pad 11: /Analog Output/BUF0_L -> /Analog Output/BUF0_R
- U9 pad 6: /Analog Output/BUF0_R -> /Analog Output/BUF0_L
- U9 pad 8: /Analog Output/F_PDM0_R -> /Analog Output/F_PDM0_L
Routing:
- net /Vout: track 0.00 -> 107.8 mm
- net VBUS: track 0.00 -> 65.0 mm, vias 0 -> 2
- net +BATT: track 0.00 -> 63.8 mm
- net -BATT: track 0.00 -> 55.1 mm
- net +3V3: track 0.00 -> 50.2 mm
- net /PSU_EN: track 0.00 -> 49.0 mm, vias 0 -> 1
- net /MII_GRXCK: track 0.00 -> 42.7 mm
- net /D+: track 0.00 -> 34.3 mm
- net /D-: track 0.00 -> 34.3 mm
- net /MII_GMDC: track 0.00 -> 30.8 mm
- net /Power Supply/!CHG: track 0.00 -> 30.0 mm, vias 0 -> 2
- net /MII_GMDIO: track 0.00 -> 30.0 mm
- net +1V2: track 12.5 -> 39.5 mm
- net /MII_GRX[3]: track 0.00 -> 26.3 mm
- net /MII_GRX[2]: track 0.00 -> 25.7 mm
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- added copper zone on In1.Cu, net GND

Commit message: Checkpoint before audio re-layout
Parts:
- added J7: Conn_02x14_Odd_Even, up5k-synth:PinHeader_2x14_P2.54mm_Vertical, F.Cu at (114.1, 123.3)
- added J8: Conn_02x05_Odd_Even, up5k-synth:PinHeader_2x05_P2.54mm_Vertical, F.Cu at (145.5, 105.6)
- moved R16 20.8 mm to (73.6, 70.2), turned to 270 degrees
- moved R17 15.8 mm to (77.2, 82.8), turned to 180 degrees
- moved R18 10.1 mm to (80.2, 73.9), turned to 180 degrees
- moved R15 6.00 mm to (84.5, 69.6), turned to 270 degrees
- moved C26 5.65 mm to (95.7, 80.8), turned to 270 degrees
- moved C9 3.79 mm to (60.4, 98.2)
- moved C8 2.02 mm to (75.8, 109.7)
- moved C10 1.70 mm to (83.1, 108.3), turned to 180 degrees
- moved C3 0.68 mm to (64.4, 99.5)
- moved C7 0.60 mm to (64.3, 97.2)
- moved C25 0.30 mm to (122.0, 92.3)
- moved C13 0.21 mm to (89.6, 97.2)
- moved C24 0.19 mm to (63.8, 92.2)
- moved C14 0.09 mm to (89.7, 101.7)
Connections:
- net /DISPLAY_CMD renamed Net-(U1-Pad22)
- net /DISPLAY_CS renamed Net-(U1-Pad21)
- net /DISPLAY_RST renamed Net-(U1-Pad23)
- net /LED_DATA renamed Net-(U1-Pad96)
- net /SEQ_LE renamed Net-(U1-Pad84)
- net /SW_CLK renamed Net-(U1-Pad79)
- net /SW_DATA renamed Net-(U1-Pad32)
- net /SW_LOAD renamed Net-(U1-Pad78)
- R15 pad 1: /SDHC1_DAT[1] -> /SDHC1_DAT[2]
- R15 pad 2: /SDHC1_DAT[0] -> /SDHC1_DAT[3]
- R15 pad 3: /SDHC1_DAT[3] -> /SDHC1_DAT[1]
- R15 pad 4: /SDHC1_DAT[2] -> /SDHC1_DAT[0]
- U1 pad 83: /SEQ_OE -> /UEXT_CS
- U1 pad 85: /SEQ_DATA -> /SC1_TXD_PAD[0]
- U1 pad 86: /SEQ_CLK -> /SC1_RXD_PAD[1]
- U2 pad 2: /MII_GTX[2] -> /MII_GTX[1]
- U2 pad 3: /MII_GTX[3] -> /MII_GTX[0]
- U2 pad 4: /MII_GRDV -> /MII_GTEN
- U2 pad 46: /MII_GTEN -> /MII_GTXER
- U2 pad 47: /MII_GTX[0] -> /MII_GTX[3]
- U2 pad 48: /MII_GTX[1] -> /MII_GTX[2]
- U2 pad 6: /MII_GTXER -> /MII_GRDV
Routing:
- net GND: track 3.00 -> 111.9 mm, vias 15 -> 79
- net /UEXT_CS: track 0.00 -> 90.9 mm, vias 0 -> 1
- net /SC4_PAD[0]: track 0.00 -> 90.3 mm, vias 0 -> 2
- net /SC0_SDA_PAD[0]: track 0.00 -> 89.9 mm, vias 0 -> 1
- net /SC1_RXD_PAD[1]: track 0.00 -> 86.9 mm, vias 0 -> 1
- net /SC0_SCL_PAD[1]: track 0.00 -> 85.9 mm, vias 0 -> 1
- net /SC4_SCK_PAD[1]: track 0.00 -> 85.0 mm, vias 0 -> 2
- net /SC4_PAD[3]: track 0.00 -> 84.0 mm, vias 0 -> 2
- net /SC1_TXD_PAD[0]: track 0.00 -> 83.5 mm, vias 0 -> 1
- net /ADC0IN[13]: track 0.00 -> 80.5 mm, vias 0 -> 1
- net /ADC0IN[12]: track 0.00 -> 78.6 mm, vias 0 -> 1
- net /ADC0IN[15]: track 0.00 -> 77.6 mm, vias 0 -> 1
- net /ADC0IN[14]: track 0.00 -> 75.8 mm, vias 0 -> 1
- net +3V3: track 50.2 -> 125.8 mm, vias 0 -> 30
- net /ADC0IN[10]: track 0.00 -> 70.1 mm, vias 0 -> 1
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- added copper zone on In2.Cu, net +3V3

Commit message: Review ready version of GF-MINUS1
Parts:
- added R10: R_100kR_0603, up5k-synth:R_0603_1608Metric_Pad0.98x0.95mm_HandSolder, B.Cu at (105.4, 124.6)
- added R11: R_100kR_0603, up5k-synth:R_0603_1608Metric_Pad0.98x0.95mm_HandSolder, B.Cu at (109.2, 123.3)
- added R3: R_100kR_0603, up5k-synth:R_0603_1608Metric_Pad0.98x0.95mm_HandSolder, B.Cu at (64.0, 97.7)
- added R5: R_100kR_0603, up5k-synth:R_0603_1608Metric_Pad0.98x0.95mm_HandSolder, B.Cu at (67.3, 97.6)
- added R6: R_100kR_0603, up5k-synth:R_0603_1608Metric_Pad0.98x0.95mm_HandSolder, B.Cu at (95.2, 75.0)
- added R7: R_100kR_0603, up5k-synth:R_0603_1608Metric_Pad0.98x0.95mm_HandSolder, B.Cu at (95.2, 69.7)
- added R8: R_100kR_0603, up5k-synth:R_0603_1608Metric_Pad0.98x0.95mm_HandSolder, B.Cu at (126.5, 80.1)
- added R9: R_100kR_0603, up5k-synth:R_0603_1608Metric_Pad0.98x0.95mm_HandSolder, B.Cu at (126.5, 76.8)
- moved R65 26.2 mm to (92.0, 70.4), turned to 180 degrees
- moved J6 23.4 mm to (123.8, 53.5), turned to 0 degrees
- moved C22 22.6 mm to (95.8, 74.2), turned to 180 degrees
- moved C33 21.7 mm to (107.6, 55.4)
- moved R80 21.7 mm to (102.2, 57.6)
- moved C37 21.7 mm to (107.7, 58.0)
- moved R82 19.1 mm to (115.2, 57.4)
- moved J5 18.9 mm to (136.2, 53.5), turned to 0 degrees
- moved U11 15.1 mm to (99.7, 63.5), turned to 270 degrees
- moved U8 13.0 mm to (98.0, 70.8), turned to 180 degrees
- moved R83 12.9 mm to (122.1, 66.2)
- moved C35 12.9 mm to (116.9, 65.5)
- moved C38 12.9 mm to (117.3, 67.8)
- moved R81 12.9 mm to (111.1, 65.8)
- moved C53 12.0 mm to (105.8, 61.6)
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Connections:
- C48 pad 1: /Analog Output/F_PDM1_R -> /Analog Output/F_PDM1_L
- C50 pad 1: /Analog Output/F_PDM1_L -> /Analog Output/F_PDM1_R
- R69 pad 1: /PDM1_R -> /PDM1_L
- R69 pad 2: /Analog Output/F_PDM1_R -> /Analog Output/F_PDM1_L
- R71 pad 1: /PDM1_L -> /PDM1_R
- R71 pad 2: /Analog Output/F_PDM1_L -> /Analog Output/F_PDM1_R
- U17 pad 11: (no net) -> GND
- U2 pad 20: Net-(U2-Pad20) -> /MII_GCRS
- U2 pad 21: /MII_GCOL -> /MII_GRXER
- U2 pad 42: /PDM1_L -> /PDM1_R
- U2 pad 43: /PDM1_R -> /PDM1_L
- U2 pad 45: /MII_GCRS -> /MII_GCOL
Routing:
- net /SC0_SDA_PAD[0]: track 89.9 -> 238.2 mm, vias 1 -> 6
- net /SC0_SCL_PAD[1]: track 85.9 -> 229.7 mm, vias 1 -> 6
- net +3V3: track 125.8 -> 207.2 mm, vias 30 -> 33
- net GND: track 111.9 -> 181.4 mm, vias 79 -> 90
- net /dbg_rst: track 0.00 -> 47.9 mm
- net /CDONE: track 0.00 -> 46.0 mm, vias 0 -> 3
- net /MII_GCOL: track 0.00 -> 42.4 mm, vias 0 -> 2
- net /MII_GTXER: track 0.00 -> 41.0 mm, vias 0 -> 2
- net +1V2: track 39.5 -> 77.4 mm, vias 0 -> 3
- net /MII_GCRS: track 0.00 -> 33.2 mm, vias 0 -> 2
- net /MII_GRXER: track 0.00 -> 31.2 mm, vias 0 -> 2
- net /CFG_RESET_B: track 0.00 -> 29.7 mm, vias 0 -> 2
- net /Analog Output/F_PDM1_L: track 7.12 -> 26.5 mm
- net /SWCLK: track 0.00 -> 17.8 mm
- net /SWO: track 0.00 -> 15.3 mm
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- added copper zone on F.Cu, net GND

Commit message: Most finish touch
Parts:
- added REF**: MountingHole_2.5mm, up5k-synth:MountingHole_2.5mm, F.Cu at (145.9, 80.5)
- added REF**: MountingHole_2.5mm, up5k-synth:MountingHole_2.5mm, F.Cu at (57.6, 56.6)
- added REF**: MountingHole_2.5mm, up5k-synth:MountingHole_2.5mm, F.Cu at (145.1, 57.1)
- added REF**: MountingHole_2.5mm, up5k-synth:MountingHole_2.5mm, F.Cu at (146.6, 145.2)
- added REF**: MountingHole_2.5mm, up5k-synth:MountingHole_2.5mm, F.Cu at (62.6, 145.2)
- moved B1 1.65 mm to (104.6, 137.7)
- moved J3 1.20 mm to (147.1, 97.9)
- moved J8 0.90 mm to (144.6, 105.6)
Routing:
- net +3V3: track 207.2 -> 201.4 mm, vias 33 -> 32
- net GND: track 181.4 -> 175.6 mm, vias 90 -> 89
- net -BATT: track 55.1 -> 53.6 mm
- net /PMOD[4]: track 40.4 -> 39.1 mm
- net /PMOD[3]: track 38.3 -> 37.1 mm
- net /PMOD[2]: track 41.6 -> 40.4 mm
- net /PMOD[1]: track 38.9 -> 37.7 mm
- net Net-(C28-Pad2): track 18.7 -> 17.6 mm
- net /SC0_SCL_PAD[1]: track 229.7 -> 228.7 mm
- net /SC0_SDA_PAD[0]: track 238.2 -> 237.2 mm
- net /SC1_RXD_PAD[1]: track 86.0 -> 85.1 mm
- net /SC4_PAD[3]: track 84.0 -> 83.1 mm
- net /SC4_SCK_PAD[1]: track 85.0 -> 84.1 mm
- net /SC1_TXD_PAD[0]: track 82.6 -> 81.7 mm
- net +BATT: track 63.8 -> 64.7 mm
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Other:
- board text added: "ANALOG"
- board text added: "GF-MINUS1 REV.A by @gatin00b"
- board text added: "PMOD"
- board text added: "RESET"
- board text added: "SD CARD"
- board text added: "SWD"
- board text added: "Thanks to alelondon, vmttmv and BlindVia for their contribution to Gluten-Free"
- board text added: "UEXT"
- board text added: "USB"
