File: hardware/boards/gluten-zero/gluten-zero.kicad_pcb (KiCad board)
At the start: 2 copper layers, 250 x 100 mm, 240 parts, among them J1 MEM2061-01-188-00-A, J2 10118194-0001LF, J3 PMOD_conn, J4 debug_conn, J5 AudioJack3_SwitchTR, J6 AudioJack3_SwitchTR, P1 keypad, P10 keypad, P11 keypad, P12 keypad, P13 keypad, P14 keypad, P15 keypad, P16 keypad, P17 keypad, P18 keypad, P19 keypad, P2 keypad, P20 keypad, P21 keypad, P22 keypad, P23 keypad, P24 keypad, P3 keypad, P4 keypad, P5 keypad, P6 keypad, P7 keypad, P8 keypad, P9 keypad, SW1 SW_Push, SW10 PB86-A2, SW11 PB86-A2, SW12 PB86-A2, SW13 PB86-A2, SW14 PB86-A2, SW15 PB86-A2, SW16 PB86-A2, SW17 PB86-A2, SW18 PB86-A2, SW19 PB86-A2, SW2 SW_Push, SW20 PB86-A2, SW21 PB86-A2, SW22 PB86-A2, SW23 PB86-A2, SW24 PB86-A2, SW25 PB86-A2, SW26 SW_DPDT_x2_MFS201N−16−Z, SW3 SW_Push, SW4 SW_Push, SW5 SW_Push, SW6 SW_Push, SW7 SW_Push, SW8 SW_Push, SW9 SW_Push, U1 ATSAME53N19A, U10 AD8531, U11 AD8531, U12 DS2745, U13 DSC6003JI2A, U14 LMS33460, U15 BQ24074, U16 TPS62120DCNR, U17 TPS63031, U18 STP16CPC26PTR, U19 STP16CPC26PTR, U2 DRA818_iCE40-UP5K-SG48, U3 74HC165, U4 74HC165, U5 74HC165, U6 74HC165, U7 DSC6003JI2A, U8 DS1881, U9 DS1881

Commit message: Scale PB86 courtyard to documented part's size
Connections:
- J3 pad 1: /PMOD[0] -> Net-(J3-Pad1)
- J3 pad 2: /PMOD[1] -> Net-(J3-Pad2)
- J3 pad 3: /PMOD[2] -> Net-(J3-Pad3)
- J3 pad 4: /PMOD[3] -> Net-(J3-Pad4)
- J3 pad 5: GND -> Net-(J3-Pad5)
- J3 pad 6: +3V3 -> Net-(J3-Pad6)
- J3 pad 7: +3V3 -> Net-(J3-Pad7)
- J3 pad 8: GND -> Net-(J3-Pad8)
- U17 pad 11: (no net) -> Net-(U17-Pad11)
